File: kicad files/gd VGC proto pcb/gd VGC proto pcb.kicad_pcb (KiCad board)
At the start: 4 copper layers, 114.3 x 73.7 mm, 121 parts, among them J1 +5V_IN, J10 VID_OUT, J11 RCA MONO OUT, J12 Main Data Bus, J13 COMSYNC, J14 Mono-Color, J15 VBL, J16 RTC, J17 RCA Shunt Select, J18 RCA, J19 CREF, J2 Video Binary B, J20 RGB In, J21 CLK_14M, J22 Memory Control, J23 VGC Extra, J24 CLK_PH0, J25 Bald-Ext-1, J26 SYNC, J27 12V_IN, J28 -5V_In, J3 Aux Data Bus, J4 DAC RGB, J5 Video Binary G, J6 COMP_RGB, J7 Video Binary R, J8 RAM Addr Bus, J9 Composite Sync, Q1 BC817, Q2 BC817, Q3 BC817, U1 MIC5504-3.3YM5, U2 28.636360 MHz

Commit message: minor silk updates before submitting
Parts:
- added REF**: KiCad-Logo_5mm_SilkScreen, Symbol:KiCad-Logo_5mm_SilkScreen, B.Cu at (120.7, 106.2)
- added REF**: OSHW-Symbol_6.7x6mm_SilkScreen, Symbol:OSHW-Symbol_6.7x6mm_SilkScreen, B.Cu at (170.8, 71.1)
- added REF**: OSHW-Symbol_6.7x6mm_SilkScreen, Symbol:OSHW-Symbol_6.7x6mm_SilkScreen, F.Cu at (150.1, 87.4)
- added svg2mod: G***, My Libraries:BE5v2, F.Cu at (114.7, 124.7)
- added svg2mod: G***, My Libraries:BE5v2, B.Cu at (155.0, 88.7)
- J16: moved to B.Cu
Other:
- board text added: "Golden Delicious VGC Proto PCB rev1.1 @baldengineer rev1"
- board text removed: "Golden Delicious VGC Proto PCB v1 @baldengineer rev1"
