File: kicad files/gd protoboard pcb/gd protoboard pcb.kicad_pcb (KiCad board)
At the start: 2 copper layers, 93.2 x 54.7 mm, 17 parts, among them J11 Addr_Main_Data, J14 CTRL2, J18 CTRL1, J6 PWR

Commit message: proto ready to fab
Parts:
- removed the C1 at (174.8, 105.9)
- removed C10, C11, C9: 1u, Capacitor_SMD:C_0805_2012Metric
- added C4: 10u, Capacitor_SMD:C_0805_2012Metric, B.Cu at (193.1, 115.1)
- added C5: 1u, Capacitor_SMD:C_0805_2012Metric, B.Cu at (196.1, 107.6)
- added C6: 1u, Capacitor_SMD:C_0805_2012Metric, B.Cu at (196.7, 101.3)
- added D4: -5v, LED_SMD:LED_1206_3216Metric, F.Cu at (196.0, 73.8)
- added J13: Conn_01x04, My Libraries:HoleField_1x05_P2.54mm, F.Cu at (188.7, 79.0)
- added J13: Conn_01x04, My Libraries:HoleField_1x05_P2.54mm, F.Cu at (176.0, 96.8)
- added J13: Conn_01x04, My Libraries:HoleField_1x05_P2.54mm, F.Cu at (168.4, 96.8)
- added J13: Conn_01x04, My Libraries:HoleField_1x05_P2.54mm, F.Cu at (170.9, 96.8)
- added J13: Conn_01x04, My Libraries:HoleField_1x05_P2.54mm, F.Cu at (183.6, 96.8)
- added J13: Conn_01x04, My Libraries:HoleField_1x05_P2.54mm, F.Cu at (181.1, 96.8)
- added J13: Conn_01x04, My Libraries:HoleField_1x05_P2.54mm, F.Cu at (165.9, 96.8)
- added J13: Conn_01x04, My Libraries:HoleField_1x05_P2.54mm, F.Cu at (158.2, 96.8)
- added J13: Conn_01x04, My Libraries:HoleField_1x05_P2.54mm, F.Cu at (153.2, 96.8)
- added J13: Conn_01x04, My Libraries:HoleField_1x05_P2.54mm, F.Cu at (127.8, 96.8)
- added J13: Conn_01x04, My Libraries:HoleField_1x05_P2.54mm, F.Cu at (148.1, 96.8)
- added J13: Conn_01x04, My Libraries:HoleField_1x05_P2.54mm, F.Cu at (173.5, 79.0)
- added J13: Conn_01x04, My Libraries:HoleField_1x05_P2.54mm, F.Cu at (143.0, 96.8)
- added J13: Conn_01x04, My Libraries:HoleField_1x05_P2.54mm, F.Cu at (140.5, 96.8)
- added J13: Conn_01x04, My Libraries:HoleField_1x05_P2.54mm, F.Cu at (132.8, 96.8)
- added J13: Conn_01x04, My Libraries:HoleField_1x05_P2.54mm, F.Cu at (117.6, 96.8)
- added J13: Conn_01x04, My Libraries:HoleField_1x05_P2.54mm, F.Cu at (115.1, 96.8)
- added J13: Conn_01x04, My Libraries:HoleField_1x05_P2.54mm, F.Cu at (150.6, 96.8)
- added J13: Conn_01x04, My Libraries:HoleField_1x05_P2.54mm, F.Cu at (155.7, 96.8)
- added J13: Conn_01x04, My Libraries:HoleField_1x05_P2.54mm, F.Cu at (130.3, 96.8)
- added J13: Conn_01x04, My Libraries:HoleField_1x05_P2.54mm, F.Cu at (145.5, 96.8)
- added J13: Conn_01x04, My Libraries:HoleField_1x05_P2.54mm, F.Cu at (122.7, 96.8)
- added J13: Conn_01x04, My Libraries:HoleField_1x05_P2.54mm, F.Cu at (188.7, 96.8)
- added J13: Conn_01x04, My Libraries:HoleField_1x05_P2.54mm, F.Cu at (160.8, 96.8)
- added J13: Conn_01x04, My Libraries:HoleField_1x05_P2.54mm, F.Cu at (125.2, 96.8)
- added J13: Conn_01x04, My Libraries:HoleField_1x05_P2.54mm, F.Cu at (120.1, 96.8)
- added J13: Conn_01x04, My Libraries:HoleField_1x05_P2.54mm, F.Cu at (110.0, 96.8)
- added J13: Conn_01x04, My Libraries:HoleField_1x05_P2.54mm, F.Cu at (137.9, 96.8)
- added J13: Conn_01x04, My Libraries:HoleField_1x05_P2.54mm, F.Cu at (112.5, 96.8)
- added J13: Conn_01x04, My Libraries:HoleField_1x05_P2.54mm, F.Cu at (183.6, 79.0)
- added J13: Conn_01x04, My Libraries:HoleField_1x05_P2.54mm, F.Cu at (181.1, 79.0)
- added J13: Conn_01x04, My Libraries:HoleField_1x05_P2.54mm, F.Cu at (178.6, 79.0)
- added J13: Conn_01x04, My Libraries:HoleField_1x05_P2.54mm, F.Cu at (176.0, 79.0)
- added J13: Conn_01x04, My Libraries:HoleField_1x05_P2.54mm, F.Cu at (186.2, 96.8)
- added J13: Conn_01x04, My Libraries:HoleField_1x05_P2.54mm, F.Cu at (170.9, 79.0)
- added J13: Conn_01x04, My Libraries:HoleField_1x05_P2.54mm, F.Cu at (168.4, 79.0)
- added J13: Conn_01x04, My Libraries:HoleField_1x05_P2.54mm, F.Cu at (165.9, 79.0)
- added J13: Conn_01x04, My Libraries:HoleField_1x05_P2.54mm, F.Cu at (163.3, 79.0)
- added J13: Conn_01x04, My Libraries:HoleField_1x05_P2.54mm, F.Cu at (158.2, 79.0)
- added J13: Conn_01x04, My Libraries:HoleField_1x05_P2.54mm, F.Cu at (155.7, 79.0)
- added J13: Conn_01x04, My Libraries:HoleField_1x05_P2.54mm, F.Cu at (153.2, 79.0)
- added J13: Conn_01x04, My Libraries:HoleField_1x05_P2.54mm, F.Cu at (150.6, 79.0)
- added J13: Conn_01x04, My Libraries:HoleField_1x05_P2.54mm, F.Cu at (148.1, 79.0)
- added J13: Conn_01x04, My Libraries:HoleField_1x05_P2.54mm, F.Cu at (145.5, 79.0)
- added J13: Conn_01x04, My Libraries:HoleField_1x05_P2.54mm, F.Cu at (186.2, 79.0)
- added J13: Conn_01x04, My Libraries:HoleField_1x05_P2.54mm, F.Cu at (143.0, 79.0)
- added J13: Conn_01x04, My Libraries:HoleField_1x05_P2.54mm, F.Cu at (140.5, 79.0)
- added J13: Conn_01x04, My Libraries:HoleField_1x05_P2.54mm, F.Cu at (137.9, 79.0)
- added J13: Conn_01x04, My Libraries:HoleField_1x05_P2.54mm, F.Cu at (160.8, 79.0)
- added J13: Conn_01x04, My Libraries:HoleField_1x05_P2.54mm, F.Cu at (132.8, 79.0)
- added J13: Conn_01x04, My Libraries:HoleField_1x05_P2.54mm, F.Cu at (130.3, 79.0)
- added J13: Conn_01x04, My Libraries:HoleField_1x05_P2.54mm, F.Cu at (127.8, 79.0)
- added J13: Conn_01x04, My Libraries:HoleField_1x05_P2.54mm, F.Cu at (125.2, 79.0)
- added J13: Conn_01x04, My Libraries:HoleField_1x05_P2.54mm, F.Cu at (122.7, 79.0)
- added J13: Conn_01x04, My Libraries:HoleField_1x05_P2.54mm, F.Cu at (120.1, 79.0)
- added J13: Conn_01x04, My Libraries:HoleField_1x05_P2.54mm, F.Cu at (135.4, 96.8)
- added J13: Conn_01x04, My Libraries:HoleField_1x05_P2.54mm, F.Cu at (117.6, 79.0)
- added J13: Conn_01x04, My Libraries:HoleField_1x05_P2.54mm, F.Cu at (115.1, 79.0)
- added J13: Conn_01x04, My Libraries:HoleField_1x05_P2.54mm, F.Cu at (112.5, 79.0)
- added J13: Conn_01x04, My Libraries:HoleField_1x05_P2.54mm, F.Cu at (110.0, 79.0)
- added J13: Conn_01x04, My Libraries:HoleField_1x05_P2.54mm, F.Cu at (135.4, 79.0)
- added J13: Conn_01x04, My Libraries:HoleField_1x05_P2.54mm, F.Cu at (178.6, 96.8)
- added J13: Conn_01x04, My Libraries:HoleField_1x05_P2.54mm, F.Cu at (173.5, 96.8)
- added J13: Conn_01x04, My Libraries:HoleField_1x05_P2.54mm, F.Cu at (163.3, 96.8)
- added J5: -5V In, Connector_PinHeader_2.54mm:PinHeader_2x02_P2.54mm_Vertical, F.Cu at (198.2, 92.3)
- added J6: PWR, Connector_PinHeader_2.54mm:PinHeader_2x04_P2.54mm_Vertical, F.Cu at (198.3, 118.9)
- added J7: CTRL2, Connector_PinHeader_2.54mm:PinHeader_2x05_P2.54mm_Vertical, F.Cu at (119.6, 118.9)
- added J8: Addr_Main_Data, Connector_PinHeader_2.54mm:PinHeader_2x16_P2.54mm_Vertical, F.Cu at (165.4, 118.9)
- added J8: Conn_01x04, My Libraries:HoleField_1x04_P2.54mm, F.Cu at (120.1, 113.3)
- added J8: Conn_01x04, My Libraries:HoleField_1x04_P2.54mm, F.Cu at (181.1, 110.7)
- added J8: Conn_01x04, My Libraries:HoleField_1x04_P2.54mm, F.Cu at (170.9, 110.7)
- added J8: Conn_01x04, My Libraries:HoleField_1x04_P2.54mm, F.Cu at (130.3, 110.7)
- added J8: Conn_01x04, My Libraries:HoleField_1x04_P2.54mm, F.Cu at (150.6, 110.7)
- added J8: Conn_01x04, My Libraries:HoleField_1x04_P2.54mm, F.Cu at (160.8, 110.7)
- added J8: Conn_01x04, My Libraries:HoleField_1x04_P2.54mm, F.Cu at (140.5, 110.7)
- added J8: Conn_01x04, My Libraries:HoleField_1x04_P2.54mm, F.Cu at (120.1, 110.7)
- added J8: Conn_01x04, My Libraries:HoleField_1x04_P2.54mm, F.Cu at (110.0, 75.2)
- added J8: Conn_01x04, My Libraries:HoleField_1x04_P2.54mm, F.Cu at (181.1, 75.2)
- added J8: Conn_01x04, My Libraries:HoleField_1x04_P2.54mm, F.Cu at (110.0, 113.3)
- added J8: Conn_01x04, My Libraries:HoleField_1x04_P2.54mm, F.Cu at (170.9, 75.2)
- added J8: Conn_01x04, My Libraries:HoleField_1x04_P2.54mm, F.Cu at (130.3, 75.2)
- added J8: Conn_01x04, My Libraries:HoleField_1x04_P2.54mm, F.Cu at (150.6, 75.2)
- added J8: Conn_01x04, My Libraries:HoleField_1x04_P2.54mm, F.Cu at (160.8, 75.2)
- added J8: Conn_01x04, My Libraries:HoleField_1x04_P2.54mm, F.Cu at (140.5, 75.2)
- added J8: Conn_01x04, My Libraries:HoleField_1x04_P2.54mm, F.Cu at (120.1, 75.2)
- added J8: Conn_01x04, My Libraries:HoleField_1x04_P2.54mm, F.Cu at (181.1, 72.6)
- added J8: Conn_01x04, My Libraries:HoleField_1x04_P2.54mm, F.Cu at (170.9, 72.6)
- added J8: Conn_01x04, My Libraries:HoleField_1x04_P2.54mm, F.Cu at (160.8, 72.6)
- added J8: Conn_01x04, My Libraries:HoleField_1x04_P2.54mm, F.Cu at (150.6, 72.6)
- added J8: Conn_01x04, My Libraries:HoleField_1x04_P2.54mm, F.Cu at (181.1, 113.3)
- added J8: Conn_01x04, My Libraries:HoleField_1x04_P2.54mm, F.Cu at (140.5, 72.6)
- added J8: Conn_01x04, My Libraries:HoleField_1x04_P2.54mm, F.Cu at (130.3, 72.6)
- added J8: Conn_01x04, My Libraries:HoleField_1x04_P2.54mm, F.Cu at (120.1, 72.6)
- added J8: Conn_01x04, My Libraries:HoleField_1x04_P2.54mm, F.Cu at (110.0, 72.6)
- added J8: Conn_01x04, My Libraries:HoleField_1x04_P2.54mm, F.Cu at (110.0, 110.7)
- added J8: Conn_01x04, My Libraries:HoleField_1x04_P2.54mm, F.Cu at (150.6, 113.3)
- added J8: Conn_01x04, My Libraries:HoleField_1x04_P2.54mm, F.Cu at (170.9, 113.3)
- added J8: Conn_01x04, My Libraries:HoleField_1x04_P2.54mm, F.Cu at (130.3, 113.3)
- added J8: Conn_01x04, My Libraries:HoleField_1x04_P2.54mm, F.Cu at (160.8, 113.3)
- added J8: Conn_01x04, My Libraries:HoleField_1x04_P2.54mm, F.Cu at (140.5, 113.3)
- added J9: CTRL1, Connector_PinHeader_2.54mm:PinHeader_2x05_P2.54mm_Vertical, F.Cu at (183.1, 118.9)
- added R4: 1k, Resistor_SMD:R_0805_2012Metric, B.Cu at (195.9, 73.8)
- added U1: L7905, Package_TO_SOT_THT:TO-220-3_Vertical, F.Cu at (198.5, 108.8)
- added svg2mod: G***, My Libraries:BE5v2, F.Cu at (166.7, 121.9)
- D1: renamed from D2; value -5v -> -12v
- moved C2 37.1 mm to (197.0, 89.9), turned to 180 degrees
- moved D3 35.0 mm to (196.0, 81.9), turned to 0 degrees
- moved R3 34.9 mm to (195.9, 81.9), turned to 0 degrees
- moved D1 32.6 mm to (196.0, 79.2), turned to 0 degrees
- moved R1 32.5 mm to (195.9, 79.2), turned to 0 degrees
- moved D2 30.3 mm to (196.0, 76.5), turned to 0 degrees
- moved R2 30.3 mm to (195.9, 76.5), turned to 0 degrees
- moved C1 10.3 mm to (188.2, 119.9)
- moved C3 7.76 mm to (195.8, 115.1)
- renumbered C6 to C1, C7 to C2, C8 to C3, D3 to D2, D4 to D3, J6 to J1, J14 to J2, J11 to J3, J18 to J4, R9 to R1, R7 to R2, R8 to R3
Connections:
- C2 pad 1: +12V -> -5V
- J2 pad 1: Net-(J14-Pad1) -> /~RDY
- J2 pad 3: Net-(J14-Pad3) -> /~NMI
- J2 pad 4: Net-(J14-Pad4) -> /KSEL0
- J2 pad 5: Net-(J14-Pad5) -> /~DMA
- J2 pad 6: Net-(J14-Pad6) -> /KSEL1
- J2 pad 8: Net-(J14-Pad8) -> /KSEL2
- J4 pad 1: Net-(J18-Pad1) -> /~IRQ
- J4 pad 3: /RESET -> /~RESET
- J4 pad 4: Net-(J18-Pad4) -> /CREF
- J4 pad 5: Net-(J18-Pad5) -> /RW
- J4 pad 7: Net-(J18-Pad7) -> /~INH
- J4 pad 8: Net-(J18-Pad8) -> /PH0
Routing:
- net (no net): track 0.00 -> 955.3 mm
- net -12V: track 0.00 -> 79.2 mm
- net +5V: track 0.00 -> 48.7 mm, vias 0 -> 2
- net GND: track 0.00 -> 40.6 mm, vias 0 -> 4
- net +12V: track 0.00 -> 39.9 mm, vias 0 -> 2
- net -5V: track 0.00 -> 28.7 mm
- net /MD0: track 0.00 -> 8.59 mm
- net /PH0: track 0.00 -> 8.45 mm
- net /MD4: track 0.00 -> 8.45 mm
- net /MD2: track 0.00 -> 8.45 mm
- net /BA6: track 0.00 -> 8.45 mm
- net /BA2: track 0.00 -> 8.45 mm
- net /BA14: track 0.00 -> 8.45 mm
- net /BA12: track 0.00 -> 8.45 mm
- net /BA0: track 0.00 -> 8.45 mm
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- added copper zone on B.Cu, net +12V
- added copper zone on F.Cu, net +12V
- added copper zone on B.Cu, net +5V
- added copper zone on F.Cu, net +5V
- added copper zone on B.Cu, net -12V
- added copper zone on F.Cu, net -12V
- added copper zone on B.Cu, net -5V
- added copper zone on B.Cu, net GND
- added copper zone on F.Cu, net GND
Other:
- board size 93.2 x 54.7 mm -> 93.2 x 64.1 mm
- board text added: "+12V"
- board text added: "+5V"
- board text added: "-12V"
- board text added: "-5"
- board text added: "-5V"
- board text added: "10"
- board text added: "15"
- board text added: "20"
- board text added: "25"
- board text added: "30"
- board text added: "5"
- board text added: "7M"
- board text added: "A"
- board text added: "A0"
- board text added: "A1"
- board text added: "A10"
- board text added: "A11"
- board text added: "A12"
- board text added: "A13"
- board text added: "A14"
- board text added: "A15"
- board text added: "A2"
- board text added: "A3"
- board text added: "A4"
- board text added: "A5"
- board text added: "A6"
- board text added: "A7"
- board text added: "A8"
- board text added: "A9"
- board text added: "B"
- board text added: "C"
- board text added: "C06"
- board text added: "CRF"
- board text added: "D"
- board text added: "D0"
- board text added: "D1"
- board text added: "D2"
- board text added: "D3"
- board text added: "D4"
- board text added: "D5"
- board text added: "D6"
- board text added: "D7"
- board text added: "E"
- board text added: "F"
- board text added: "G"
- board text added: "H"
- board text added: "I"
- board text added: "J"
- board text added: "K0"
- board text added: "K1"
- board text added: "K2"
- board text added: "PH0"
- board text added: "Q3"
- board text added: "RW"
- board text added: "gd Protoboard Rev1 ● 2021-09-08 ● @baldengineer"
- board text added: "~DMA"
- board text added: "~INH"
- board text added: "~IRQ"
- board text added: "~NMI"
- board text added: "~RDY"
- board text added: "~RES"
- board text removed: "BA0 BA1"
- board text removed: "BA10 BA11"
- board text removed: "BA14 BA15"
- board text removed: "BA6 BA7"
- board text removed: "MD1"
- board text removed: "MD5"
