File: kicad files/gd rp2040 keyboard proto pcb/kicad/gd rp2040 keyboard proto pcb.kicad_pcb (KiCad board)
At the start: 2 copper layers, 79.2 x 49.5 mm, 64 parts, among them J1 USB Pwr, J10 CTRL1-HDR, J11 CTRL2-HDR, J12 USB_A, J13 3v3, J13 Conn_01x04, J14 GPIO, J15 ADC, J2 Conn_01x02, J3 Power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

Commit message: parial route of rev2
Parts:
- removed the J13 at (93.2, 92.4)
- removed the J13 at (95.7, 92.4)
- removed the J13 at (90.6, 105.1)
- removed the J13 at (88.1, 105.1)
- removed the J13 at (85.5, 105.1)
- removed the J13 at (83.0, 105.1)
- removed the J13 at (83.0, 92.4)
- removed the J13 at (85.5, 92.4)
- removed the J13 at (88.1, 92.4)
- removed the J13 at (90.6, 92.4)
- removed J15: ADC, Connector_PinHeader_2.54mm:PinHeader_2x03_P2.54mm_Vertical
- removed J8 (x3): Conn_01x04, My Libraries:HoleField_1x04_P2.54mm
- removed J8: VUSB Break Outs, Connector_PinSocket_2.54mm:PinSocket_1x03_P2.54mm_Vertical
- removed REF**: OSHW-Symbol_6.7x6mm_SilkScreen, Symbol:OSHW-Symbol_6.7x6mm_SilkScreen
- removed REF** (x2): KiCad-Logo2_5mm_Copper, Symbol:KiCad-Logo2_5mm_Copper
- removed RNP1: 10k, Resistor_SMD:R_0805_2012Metric
- removed RNP2: 10K, Resistor_SMD:R_0805_2012Metric
- removed svg2mod: G***, My Libraries:BE5v2
- added Ctx1: 100n, Capacitor_SMD:C_0603_1608Metric, B.Cu at (130.4, 112.0)
- added Ctx2: 100n, Capacitor_SMD:C_0603_1608Metric, B.Cu at (130.5, 117.8)
- added R10: 4k7, Resistor_SMD:R_0805_2012Metric, B.Cu at (93.9, 98.1)
- added R9: 4k7, Resistor_SMD:R_0805_2012Metric, B.Cu at (105.4, 108.2)
- added Rdnp1: 4k7, Resistor_SMD:R_0805_2012Metric, B.Cu at (127.8, 115.2)
- added SW2: MEGA POWER, My Libraries:SW_Push_CK_PTS525_SM15, F.Cu at (73.2, 99.7)
- added U5: TXB0108PW, Package_SO:TSSOP-20_4.4x6.5mm_P0.65mm, F.Cu at (129.3, 114.9)
- J2: value Conn_01x02 -> Power Sequence; footprint Connector_PinHeader_2.54mm:PinHeader_1x02_P2.54mm_Vertical -> Connector_PinSocket_2.54mm:PinSocket_1x05_P2.54mm_Vertical
- R1: value 1k -> 4k7; moved to B.Cu
- SW1: value RUN-VERIFY FOOTPRINT -> 2040 RESET
- Y1: value ABLS-12.000MHZ-B4-T -> ECS-120-18-33-JEM-TR; footprint RP2040_minimal:Crystal_SMD_HC49-US -> Crystal:Crystal_SMD_3225-4Pin_3.2x2.5mm
- moved J2 40.0 mm to (141.1, 90.8)
- moved R1 27.6 mm to (127.0, 112.0), turned to 180 degrees
- moved U4 11.5 mm to (89.7, 105.8), turned to 0 degrees
- moved U2 9.45 mm to (106.3, 92.6)
- moved SW1 2.46 mm to (67.6, 99.7), turned to 270 degrees
Connections:
- J14 pad 13: /GPIO25 -> GND
- J2 pad 1: /~USB_BOOT -> GND
- J2 pad 2: GND -> /MEGA_POWER
- J7 pad 11: Net-(J7-Pad11) -> GND
- R1 pad 1: /QSPI_SS -> +3V3
- R1 pad 2: /~USB_BOOT -> /TXen
- U3 pad 11: /D3 -> /D5
- U3 pad 12: /D2 -> /D6
- U3 pad 13: /D1 -> /D7
- U3 pad 14: /D0 -> /245_EN
- U3 pad 15: /245_EN -> /RESETrp
- U3 pad 16: /GPIO13 -> /KSEL1rp
- U3 pad 17: /GPIO14 -> /KSEL2rp
- U3 pad 18: /GPIO15 -> /RWrp
- U3 pad 27: /GPIO16 -> /PH0rp
- U3 pad 37: /GPIO25 -> /TXen
- U3 pad 38: /GPIO26_ADC0 -> /MEGA_POWER
- U3 pad 39: /GPIO27_ADC1 -> /-12V_Enable
- U3 pad 4: /VBUS-En -> /KSEL0rp
- U3 pad 40: /GPIO28_ADC2 -> /+12V_Enable
- U3 pad 41: /GPIO29_ADC3 -> /+5V_Enable
- U3 pad 5: /VBUS-OC -> /D0
- U3 pad 6: /VBUS-Detect -> /D1
- U3 pad 7: /D6 -> /D2
- U3 pad 8: /D5 -> /D3
- U4 pad 1: +5V -> Net-(R9-Pad2)
- U4 pad 11: Net-(U4-Pad11) -> /MD7
- U4 pad 9: +5V -> /D7
- Y1 pad 2: Net-(C3-Pad1) -> GND
Routing:
- net /QSPI_SCLK: track 42.3 -> 12.3 mm, vias 2 -> 0
- net /D3: track 29.3 -> 0.00 mm, vias 2 -> 0
- net /QSPI_SD3: track 41.9 -> 13.5 mm, vias 2 -> 0
- net /MEGA_POWER: track 0.00 -> 28.3 mm
- net /D6: track 27.4 -> 0.00 mm, vias 2 -> 0
- net /QSPI_SD0: track 39.1 -> 11.9 mm
- net /D2: track 26.3 -> 0.00 mm, vias 2 -> 0
- net /D5: track 24.8 -> 0.00 mm, vias 2 -> 0
- net /GPIO27_ADC1: track 24.2 -> 0.00 mm
- net /D4: track 23.2 -> 0.00 mm, vias 2 -> 0
- net /245_EN: track 22.9 -> 0.00 mm, vias 2 -> 0
- net /GPIO26_ADC0: track 22.8 -> 0.00 mm
- net /GPIO29_ADC3: track 20.5 -> 0.00 mm
- net /GPIO25: track 19.6 -> 0.00 mm
- net /-12V_Enable: track 0.00 -> 19.4 mm
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Other:
- board text added: "gd rp2040/kbd 2021-10-22 r2 @baldengineer"
- board text removed: "DET"
- board text removed: "En"
- board text removed: "J8"
- board text removed: "OC"
- board text removed: "USB Boot"
- board text removed: "USB..."
- board text removed: "gd rp2040/kbd 2021-09-06 r1 @baldengineer"
