File: kicad files/gd rev3/mega-6502.kicad_sch (KiCad schematic)
At the start: 50 parts, among them J1 XY, Q1 BC817, Q2 BC817, SW1 RESET, U1 74HC02-CHECK FOOTPRINT, U10 DRAM64KX4, U2 w65c02s, U3 Apple_MEGA_II, U4 74HCT245, U5 74HCT245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

Commit message: poking around with the laying
Parts:
- removed C6: 100uF, Capacitor_Tantalum_SMD:CP_EIA-3216-18_Kemet-A_Pad1.58x1.35mm_HandSolder, symbol Device:CP
- added C54: 1uF, Capacitor_SMD:C_0805_2012Metric, symbol Device:C_Small
- added R47: 470, Resistor_SMD:R_0805_2012Metric, symbol My_Library:R_0805
Connections:
- net INT_14M is gone; now on net 14M: X1.3 (OUT)
- net +5V: now also C54.1
- net GND: now also C54.2
- net ~{ROMEN}: no longer R7.2
- net at D1.1 (K): now also R47.1; no longer Q1.3 (C)
- new net: Q1.3 (C), R47.2
Other:
- moved on the sheet: D1, Q1, R7

Commit message: extended mega-65c02 sheet
Connections:
- net ~{ROMEN}: now also R7.2
- net C060-67 renamed ~{C060-67}
- net CASA renamed ~{CASA}
- net CASA.B renamed ~{CASA.B}
- net CASM renamed ~{CASM}
- net CASM.B renamed ~{CASM.B}
- net KSEL1 renamed ~{KSEL1}
- net KSEL2 renamed ~{KSEL2}
- net PDLTRIG renamed ~{PDLTRIG}
- net RAMWE renamed ~{RAMWE}
- net RAS renamed ~{RAS}
- net RAS.B renamed ~{RAS.B}
- net RWE.B renamed ~{RWE.B}
- net WINDOW renamed ~{WINDOW}
Other:
- moved on the sheet: C10, C11, C8, C9, RN1, RN2, RN3, U10, U1A, U7, U8, U9

Commit message: after crash commit. arranging high-level sheet signals (and added audio circuit)
Parts:
- removed BZ1: Buzzer, My Libraries:12mm_Piezo_Buzzer, symbol Device:Buzzer
- removed C5: 100nF, Capacitor_SMD:C_0805_2012Metric, symbol Device:C
- removed D2: SNDZ, LED_SMD:LED_1206_3216Metric, symbol My_Library:D_1206
- removed Q2: BC817, Package_TO_SOT_SMD:SOT-23, symbol Device:Q_NPN_BEC
- removed R10: 1k, Resistor_SMD:R_0805_2012Metric, symbol My_Library:R_0805
- removed R8: 220, Resistor_SMD:R_0805_2012Metric, symbol My_Library:R_0805
- removed R9: 10k, Resistor_SMD:R_0805_2012Metric, symbol My_Library:R_0805
- added C5: 100u, Capacitor_Tantalum_SMD:CP_EIA-3216-18_Kemet-A, symbol Device:C_Polarized_Small
- added C63: 1uF, Capacitor_SMD:C_0805_2012Metric, symbol Device:C_Small
- added unit 5 of U3
- renumbered U3 to U1, U1 to U3
Connections:
- net +5V: now also C5.1, C63.1, U3.14 (VCC)
- net GND: now also C5.2, C63.2, U3.7 (GND)
Other:
- title: (none) -> Mega-II 65C02
- moved on the sheet: C4, U3A

Commit message: top-level arragements, many more works to do
Connections:
- net SERVIDEO renamed SERVID
Changed lines of the file:
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@@
     (effects (font (size 1.27 1.27)) (justify right bottom))
   )
-  (label "SERVIDEO" (at 158.75 101.6 180)
+  (label "SERVID" (at 158.75 101.6 180)
     (effects (font (size 1.27 1.27)) (justify right bottom))
   )
@@
     (effects (font (size 1.27 1.27)) (justify left bottom))
   )
-  (label "SERVIDEO" (at 40.64 237.49 180)
+  (label "SERVID" (at 40.64 237.49 180)
     (effects (font (size 1.27 1.27)) (justify right bottom))
   )
@@
     (effects (font (size 1.27 1.27)) (justify right))
   )
-  (hierarchical_label "SERVIDEO" (shape input) (at 30.48 237.49 180)
-    (effects (font (size 1.27 1.27)) (justify right))
-  )
+  (hierarchical_label "SERVID" (shape input) (at 30.48 237.49 180)
+    (effects (font (size 1.27 1.27)) (justify right))
+  )

Commit message: ERC clean-up, wow, intern really messed up the symbols
Changed lines of the file:
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@@
     (stroke (width 0) (type default) (color 0 0 0 0))
   )
-  (wire (pts (xy 41.91 161.29) (xy 34.29 161.29))
-    (stroke (width 0) (type default) (color 0 0 0 0))
-  )
   (wire (pts (xy 39.37 100.33) (xy 34.29 100.33))
     (stroke (width 0) (type default) (color 0 0 0 0))
@@
     (effects (font (size 1.27 1.27)) (justify left bottom))
   )
-  (label "14M" (at 41.91 161.29 180)
-    (effects (font (size 1.27 1.27)) (justify right bottom))
-  )
   (label "BA2" (at 34.29 90.17 0)
     (effects (font (size 1.27 1.27)) (justify left bottom))
@@
     (effects (font (size 1.27 1.27)) (justify right))
   )
-  (hierarchical_label "14M" (shape input) (at 34.29 161.29 180)
-    (effects (font (size 1.27 1.27)) (justify right))
-  )
   (hierarchical_label "SERVID" (shape input) (at 30.48 237.49 180)
     (effects (font (size 1.27 1.27)) (justify right))
@@
     (pin "1")
   )
-  (symbol (lib_id "Apple_IIgs_Symbols:74HCT245") (at 153.67 186.69 0) (unit 1)
+  (symbol (lib_name "74HCT245_1") (lib_id "Apple_IIgs_Symbols:74HCT245") (at 153.67 186.69 0) (unit 1)
     (in_bom yes) (on_board yes)
     (property "Reference" "U4" (id 0) (at 156.21 167.64 0))
@@
   (symbol (lib_id "Jumper:SolderJumper_3_Open") (at 312.42 227.33 90) (unit 1)
     (in_bom yes) (on_board yes) (fields_autoplaced)
-    (property "Reference" "JP1" (id 0) (at 309.88 226.0599 90)
+    (property "Reference" "JP1" (id 0) (at 314.96 228.6001 90)
       (effects (font (size 1.27 1.27)) (justify left))
     )
-    (property "Value" "X_EN" (id 1) (at 309.88 228.5999 90)
+    (property "Value" "X_EN" (id 1) (at 314.96 226.0601 90)
       (effects (font (size 1.27 1.27)) (justify left))
     )
-    (property "Footprint" "Jumper:SolderJumper-3_P1.3mm_Open_RoundedPad1.0x1.5mm" (id 2) (at 312.42 227.33 0)
+    (property "Footprint" "Jumper:SolderJumper-3_P1.3mm_Open_RoundedPad1.0x1.5mm" (id 2) (at 312.42 233.68 0)
       (effects (font (size 1.27 1.27)) hide)
     )
@@
       (effects (font (size 1.27 1.27)) hide)
     )
-    (property "MFN" "940-44-084-24-000000" (id 4) (at 127 88.9 0)
+    (property "MFN" "940-44-084-24-000000" (id 4) (at 128.27 91.44 0)
       (effects (font (size 1.27 1.27)) hide)
     )
@@
     (pin "3")
   )
+  (symbol (lib_name "74HCT245_1") (lib_id "Apple_IIgs_Symbols:74HCT245") (at 153.67 240.03 0) (unit 1)
+    (in_bom yes) (on_board yes)
+    (property "Reference" "U5" (id 0) (at 156.21 220.98 0))
+    (property "Value" "74HCT245" (id 1) (at 160.02 223.52 0))
+    (property "Footprint" "Package_SO:SOIC-20W_7.5x12.8mm_P1.27mm" (id 2) (at 148.59 223.52 0)
+      (effects (font (size 1.27 1.27)) hide)
+    )
+    (property "Datasheet" "" (id 3) (at 148.59 223.52 0)
+      (effects (font (size 1.27 1.27)) hide)
+    )
+    (pin "1")
+    (pin "10")
+    (pin "11")
+    (pin "12")
+    (pin "13")
+    (pin "14")
+    (pin "15")
+    (pin "16")
+    (pin "17")
+    (pin "18")
+    (pin "19")
+    (pin "2")
+    (pin "20")
+    (pin "3")
+    (pin "4")
+    (pin "5")
+    (pin "6")
+    (pin "7")
+    (pin "8")
+    (pin "9")
+  )
   (symbol (lib_id "power:GND") (at 163.83 204.47 0) (unit 1)
     (in_bom yes) (on_board yes)
@@
     (pin "1")
   )
-  (symbol (lib_id "Apple_IIgs_Symbols:74HCT245") (at 153.67 240.03 0) (unit 1)
-    (in_bom yes) (on_board yes)
-    (property "Reference" "U5" (id 0) (at 156.21 219.71 0))
-    (property "Value" "74HCT245" (id 1) (at 160.02 222.25 0))
-    (property "Footprint" "Package_SO:SOIC-20W_7.5x12.8mm_P1.27mm" (id 2) (at 148.59 223.52 0)
-      (effects (font (size 1.27 1.27)) hide)
-    )
-    (property "Datasheet" "" (id 3) (at 148.59 223.52 0)
-      (effects (font (size 1.27 1.27)) hide)
-    )
-    (pin "1")
-    (pin "10")
-    (pin "11")
-    (pin "12")
-    (pin "13")
-    (pin "14")
-    (pin "15")
-    (pin "16")
-    (pin "17")
-    (pin "18")
-    (pin "19")
-    (pin "2")
-    (pin "20")
-    (pin "3")
-    (pin "4")
-    (pin "5")
-    (pin "6")
-    (pin "7")
-    (pin "8")
-    (pin "9")
-  )
   (symbol (lib_id "power:GND") (at 251.46 276.86 0) (unit 1)
     (in_bom yes) (on_board yes)
@@
     (property "Reference" "U2" (id 0) (at 97.79 171.45 0))
     (property "Value" "w65c02s" (id 1) (at 100.33 173.99 0))
-    (property "Footprint" "Package_QFP:TQFP-44_10x10mm_P0.8mm" (id 2) (at 88.9 177.8 0)
+    (property "Footprint" "Package_QFP:TQFP-44_10x10mm_P0.8mm" (id 2) (at 90.17 166.37 0)
       (effects (font (size 1.27 1.27)) hide)
     )

Commit message: added missing Flash to 2040 circuits and sync'd title blocks
Other:
- company: (none) -> twitch.tv/baldengineer
Changed lines of the file:
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@@
     (title "Mega-II 65C02")
     (rev "3a")
+    (company "twitch.tv/baldengineer")
   )
   (junction (at 326.39 219.71) (diameter 0) (color 0 0 0 0)
