File: kicad files/gd rev3/Audio.kicad_sch (KiCad schematic)
At the start: 18 parts, among them J19 SPKR, J20 Ears, Q2 BC817, U26 MCP4541T, U27 LM4875

Commit message: added missing Flash to 2040 circuits and sync'd title blocks
Other:
- company: (none) -> twitch.tv/baldengineer
Changed lines of the file:
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@@
     (title "Audio")
     (rev "3a")
+    (company "twitch.tv/baldengineer")
   )
   (junction (at 198.12 101.6) (diameter 0) (color 0 0 0 0)

Commit message: on-stream clean-up work
Parts:
- J20: footprint Connector_Audio:Jack_3.5mm_PJ311_Horizontal -> My Libraries:Jack_3.5mm_tensility_54-00177
Other:
- note removed: "* DOUBLE DOUBLE CHECK THE EARPHONE PINOUT!!!"
Changed lines of the file:
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@@
     (stroke (width 0) (type default) (color 0 0 0 0))
-  )
-  (text "* DOUBLE DOUBLE CHECK THE EARPHONE PINOUT!!!" (at 67.31 52.07 0)
-    (effects (font (size 3.81 3.81)) (justify left bottom))
   )
   (text "RNP is for external drain\nresistor for 100uF cap." (at 170.18 113.03 0)
@@
       (effects (font (size 1.27 1.27)) (justify right))
     )
-    (property "Footprint" "Connector_Audio:Jack_3.5mm_PJ311_Horizontal" (id 2) (at 219.71 92.71 0)
+    (property "Footprint" "My Libraries:Jack_3.5mm_tensility_54-00177" (id 2) (at 219.71 92.71 0)
       (effects (font (size 1.27 1.27)) hide)
     )
@@
   (symbol (lib_id "My_Library:R_0805") (at 93.98 133.35 180) (unit 1)
     (in_bom yes) (on_board yes)
-    (property "Reference" "R48" (id 0) (at 97.79 134.62 0)
-      (effects (font (size 1.27 1.27)) (justify left))
-    )
+    (property "Reference" "R48" (id 0) (at 99.06 134.62 0)
+      (effects (font (size 1.27 1.27)) (justify left))
+    )

Commit message: ERC clean-up
Other:
- note added: "Are we scaling the audio on demo board?"
Changed lines of the file:
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@@
     (stroke (width 0) (type default) (color 0 0 0 0))
+  )
+  (text "Are we scaling the audio on demo board?" (at 25.4 129.54 0)
+    (effects (font (size 1.27 1.27)) (justify left bottom))
   )
   (text "RNP is for external drain\nresistor for 100uF cap." (at 170.18 113.03 0)
@@
     (effects (font (size 1.27 1.27)) (justify right bottom))
   )
-  (label "WOZ_AUD" (at 50.8 101.6 180)
-    (effects (font (size 1.27 1.27)) (justify right bottom))
-  )
   (label "Vo1" (at 182.88 90.17 180)
     (effects (font (size 1.27 1.27)) (justify right bottom))
@@
     (effects (font (size 1.27 1.27)) (justify right))
   )
-  (symbol (lib_id "My_Library:R_0805") (at 52.07 116.84 0) (unit 1)
+  (symbol (lib_name "R_0805_1") (lib_id "My_Library:R_0805") (at 52.07 116.84 0) (unit 1)
     (in_bom yes) (on_board yes)
     (property "Reference" "R9" (id 0) (at 49.53 116.84 0))
@@
     (pin "1")
   )
-  (symbol (lib_id "My_Library:R_0805") (at 198.12 96.52 0) (unit 1)
+  (symbol (lib_name "R_0805_3") (lib_id "My_Library:R_0805") (at 198.12 96.52 0) (unit 1)
     (in_bom yes) (on_board yes)
     (property "Reference" "R50" (id 0) (at 195.58 95.25 0))
@@
     (pin "1")
   )
-  (symbol (lib_id "My_Library:R_0805") (at 52.07 109.22 0) (unit 1)
+  (symbol (lib_name "R_0805_2") (lib_id "My_Library:R_0805") (at 52.07 109.22 0) (unit 1)
     (in_bom yes) (on_board yes)
     (property "Reference" "R8" (id 0) (at 49.53 109.22 0))
@@
   (symbol (lib_id "My_Library:AudioJack3_SwitchTR-Tensility_Pins") (at 219.71 92.71 180) (unit 1)
     (in_bom yes) (on_board yes)
-    (property "Reference" "J20" (id 0) (at 219.71 78.74 0)
+    (property "Reference" "J20" (id 0) (at 219.71 106.68 0)
       (effects (font (size 1.27 1.27)) (justify right))
     )
-    (property "Value" "Ears" (id 1) (at 218.44 81.28 0)
+    (property "Value" "Ears" (id 1) (at 220.98 104.14 0)
       (effects (font (size 1.27 1.27)) (justify right))
     )
-    (property "Footprint" "My Libraries:Jack_3.5mm_tensility_54-00177" (id 2) (at 219.71 92.71 0)
-      (effects (font (size 1.27 1.27)) hide)
-    )
-    (property "Datasheet" "https://tensility.s3.amazonaws.com/uploads/pdffiles/54-00178.pdf" (id 3) (at 219.71 92.71 0)
-      (effects (font (size 1.27 1.27)) hide)
-    )
-    (property "MFG" "Tensility International Corp" (id 4) (at 219.71 92.71 0)
-      (effects (font (size 1.27 1.27)) hide)
-    )
-    (property "MPN" "54-00178" (id 5) (at 219.71 92.71 0)
+    (property "Footprint" "My Libraries:Jack_3.5mm_tensility_54-00177" (id 2) (at 218.44 80.01 0)
+      (effects (font (size 1.27 1.27)) hide)
+    )
+    (property "Datasheet" "https://tensility.s3.amazonaws.com/uploads/pdffiles/54-00178.pdf" (id 3) (at 218.44 74.93 0)
+      (effects (font (size 1.27 1.27)) hide)
+    )
+    (property "MFG" "Tensility International Corp" (id 4) (at 219.71 77.47 0)
+      (effects (font (size 1.27 1.27)) hide)
+    )
+    (property "MPN" "54-00178" (id 5) (at 219.71 97.79 0)
       (effects (font (size 1.27 1.27)) hide)
     )
@@
     (pin "1")
   )
-  (symbol (lib_id "My_Library:R_0805") (at 130.81 118.11 180) (unit 1)
+  (symbol (lib_name "R_0805_5") (lib_id "My_Library:R_0805") (at 130.81 118.11 180) (unit 1)
     (in_bom yes) (on_board yes)
     (property "Reference" "R49" (id 0) (at 134.62 119.38 0))
@@
     (pin "8")
   )
-  (symbol (lib_id "My_Library:R_0805") (at 93.98 133.35 180) (unit 1)
+  (symbol (lib_name "R_0805_6") (lib_id "My_Library:R_0805") (at 93.98 133.35 180) (unit 1)
     (in_bom yes) (on_board yes)
     (property "Reference" "R48" (id 0) (at 99.06 134.62 0)
@@
     (pin "2")
   )
-  (symbol (lib_id "My_Library:R_0805") (at 173.99 95.25 0) (unit 1)
+  (symbol (lib_name "R_0805_4") (lib_id "My_Library:R_0805") (at 173.99 95.25 0) (unit 1)
     (in_bom yes) (on_board yes)
     (property "Reference" "RNP3" (id 0) (at 171.45 92.71 0))

Commit message: first pass
Parts:
- C58, C60, C61: footprint Resistor_SMD:R_0805_2012Metric -> Capacitor_SMD:C_0805_2012Metric
Changed lines of the file:
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@@
       (effects (font (size 1.27 1.27)) (justify left))
     )
-    (property "Footprint" "Resistor_SMD:R_0805_2012Metric" (id 2) (at 97.79 68.58 0)
+    (property "Footprint" "Capacitor_SMD:C_0805_2012Metric" (id 2) (at 97.79 68.58 0)
       (effects (font (size 1.27 1.27)) hide)
     )
@@
       (effects (font (size 1.27 1.27)) (justify left))
     )
-    (property "Footprint" "Resistor_SMD:R_0805_2012Metric" (id 2) (at 125.73 102.87 0)
+    (property "Footprint" "Capacitor_SMD:C_0805_2012Metric" (id 2) (at 125.73 102.87 0)
       (effects (font (size 1.27 1.27)) hide)
     )
@@
       (effects (font (size 1.27 1.27)) (justify left))
     )
-    (property "Footprint" "Resistor_SMD:R_0805_2012Metric" (id 2) (at 158.75 73.66 0)
+    (property "Footprint" "Capacitor_SMD:C_0805_2012Metric" (id 2) (at 158.75 73.66 0)
       (effects (font (size 1.27 1.27)) hide)
     )
