File: kicad files/gd power supply board pcb/gd power supply board pcb.kicad_sch (KiCad schematic)
At the start: 19 parts, among them J1 15V_IN, J2 15V_IN, J3 Edge Connector, Q1 FDS9435A

Commit message: minor fixes and compacting the floorplan. stacked 5V supplies for maximum minimage.
Parts:
- added H1, H2, H3, H4: MountingHole, MountingHole:MountingHole_2.2mm_M2, symbol Mechanical:MountingHole
- added TP3: TestPoint_Harwin, My Libraries:Harwin-S1751-46-Test-Point, symbol My Library:TestPoint_Harwin
Connections:
- net 15v_In is gone; now on net 15v_Raw: R8.2
- net Vin: now also TP3.1
Changed lines of the file:
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@@
-    (effects (font (size 1.27 1.27)) (justify right bottom))
-  )
-  (label "15v_In" (at 195.58 118.11 270)
     (effects (font (size 1.27 1.27)) (justify right bottom))
   )
@@
     (effects (font (size 1.27 1.27)) (justify left bottom))
   )
+  (label "15v_Raw" (at 195.58 118.11 270)
+    (effects (font (size 1.27 1.27)) (justify right bottom))
+  )
   (symbol (lib_id "My Library:R_0805") (at 217.17 133.35 180) (unit 1)
     (in_bom yes) (on_board yes) (fields_autoplaced)
@@
     )
     (pin "1")
+  )
+  (symbol (lib_id "Mechanical:MountingHole") (at 99.06 181.61 0) (unit 1)
+    (in_bom yes) (on_board yes) (fields_autoplaced)
+    (property "Reference" "H2" (id 0) (at 101.6 180.3399 0)
+      (effects (font (size 1.27 1.27)) (justify left))
+    )
+    (property "Value" "MountingHole" (id 1) (at 101.6 182.8799 0)
+      (effects (font (size 1.27 1.27)) (justify left))
+    )
+    (property "Footprint" "MountingHole:MountingHole_2.2mm_M2" (id 2) (at 99.06 181.61 0)
+      (effects (font (size 1.27 1.27)) hide)
+    )
+    (property "Datasheet" "~" (id 3) (at 99.06 181.61 0)
+      (effects (font (size 1.27 1.27)) hide)
+    )
   )
   (symbol (lib_id "Transistor_FET:FDS9435A") (at 77.47 133.35 90) (unit 1)
@@
     )
     (pin "1")
+  )
+  (symbol (lib_id "Mechanical:MountingHole") (at 99.06 175.26 0) (unit 1)
+    (in_bom yes) (on_board yes) (fields_autoplaced)
+    (property "Reference" "H1" (id 0) (at 101.6 173.9899 0)
+      (effects (font (size 1.27 1.27)) (justify left))
+    )
+    (property "Value" "MountingHole" (id 1) (at 101.6 176.5299 0)
+      (effects (font (size 1.27 1.27)) (justify left))
+    )
+    (property "Footprint" "MountingHole:MountingHole_2.2mm_M2" (id 2) (at 99.06 175.26 0)
+      (effects (font (size 1.27 1.27)) hide)
+    )
+    (property "Datasheet" "~" (id 3) (at 99.06 175.26 0)
+      (effects (font (size 1.27 1.27)) hide)
+    )
   )
   (symbol (lib_id "My Library:D_1206") (at 63.5 143.51 270) (unit 1)
@@
     (pin "9")
   )
+  (symbol (lib_id "Mechanical:MountingHole") (at 107.95 181.61 0) (unit 1)
+    (in_bom yes) (on_board yes) (fields_autoplaced)
+    (property "Reference" "H4" (id 0) (at 110.49 180.3399 0)
+      (effects (font (size 1.27 1.27)) (justify left))
+    )
+    (property "Value" "MountingHole" (id 1) (at 110.49 182.8799 0)
+      (effects (font (size 1.27 1.27)) (justify left))
+    )
+    (property "Footprint" "MountingHole:MountingHole_2.2mm_M2" (id 2) (at 107.95 181.61 0)
+      (effects (font (size 1.27 1.27)) hide)
+    )
+    (property "Datasheet" "~" (id 3) (at 107.95 181.61 0)
+      (effects (font (size 1.27 1.27)) hide)
+    )
+  )
   (symbol (lib_id "Connector:Barrel_Jack_Switch") (at 38.1 127 0) (mirror y) (unit 1)
     (in_bom yes) (on_board yes) (fields_autoplaced)
@@
     (pin "2")
   )
+  (symbol (lib_id "Mechanical:MountingHole") (at 107.95 175.26 0) (unit 1)
+    (in_bom yes) (on_board yes) (fields_autoplaced)
+    (property "Reference" "H3" (id 0) (at 110.49 173.9899 0)
+      (effects (font (size 1.27 1.27)) (justify left))
+    )
+    (property "Value" "MountingHole" (id 1) (at 110.49 176.5299 0)
+      (effects (font (size 1.27 1.27)) (justify left))
+    )
+    (property "Footprint" "MountingHole:MountingHole_2.2mm_M2" (id 2) (at 107.95 175.26 0)
+      (effects (font (size 1.27 1.27)) hide)
+    )
+    (property "Datasheet" "~" (id 3) (at 107.95 175.26 0)
+      (effects (font (size 1.27 1.27)) hide)
+    )
+  )
   (symbol (lib_id "power:GND") (at 77.47 147.32 0) (unit 1)
     (in_bom yes) (on_board yes) (fields_autoplaced)
@@
     )
     (property "Datasheet" "" (id 3) (at 217.17 146.05 0)
+      (effects (font (size 1.27 1.27)) hide)
+    )
+    (pin "1")
+  )
+  (symbol (lib_id "My Library:TestPoint_Harwin") (at 88.9 130.81 0) (unit 1)
+    (in_bom yes) (on_board yes) (fields_autoplaced)
+    (property "Reference" "TP3" (id 0) (at 91.44 127.5079 0)
+      (effects (font (size 1.27 1.27)) (justify left))
+    )
+    (property "Value" "TestPoint_Harwin" (id 1) (at 88.9 125.73 0)
+      (effects (font (size 1.27 1.27)) hide)
+    )
+    (property "Footprint" "My Libraries:Harwin-S1751-46-Test-Point" (id 2) (at 93.98 130.81 0)
+      (effects (font (size 1.27 1.27)) hide)
+    )
+    (property "Datasheet" "~" (id 3) (at 93.98 130.81 0)
       (effects (font (size 1.27 1.27)) hide)
     )
@@
       (reference "D9") (unit 1) (value "Rev_LED") (footprint "LED_SMD:LED_1206_3216Metric")
     )
-    (path "/2a737751-d85e-4f05-8aec-b659f83530c3/04e98119-a4c0-49e3-99b5-e1868729b021"
+    (path "/285cc15f-cf9c-424b-a5cd-4cbb5f4c72f8"
       (reference "H1") (unit 1) (value "MountingHole") (footprint "MountingHole:MountingHole_2.2mm_M2")
     )
-    (path "/2a737751-d85e-4f05-8aec-b659f83530c3/671a0fbd-386d-4717-97ea-a79816778d1b"
+    (path "/0970c0c6-ef87-4c89-ac5d-4b35bf51f93b"
       (reference "H2") (unit 1) (value "MountingHole") (footprint "MountingHole:MountingHole_2.2mm_M2")
     )
-    (path "/2a737751-d85e-4f05-8aec-b659f83530c3/d10ac24d-2358-478e-8a6c-1ddee3732a42"
+    (path "/981034d3-4ba9-410a-8568-6651f93125bb"
       (reference "H3") (unit 1) (value "MountingHole") (footprint "MountingHole:MountingHole_2.2mm_M2")
     )
-    (path "/2a737751-d85e-4f05-8aec-b659f83530c3/9a67b314-542c-4141-bf4e-677ee16eae7a"
+    (path "/357d4381-714a-4aae-aa1a-b6d69a3491ea"
       (reference "H4") (unit 1) (value "MountingHole") (footprint "MountingHole:MountingHole_2.2mm_M2")
-    )
-    (path "/fc065b92-de59-4c29-93b4-0f722018f063/6ec0f968-82bd-4a3a-bf56-0cfd68c3ad16"
-      (reference "H5") (unit 1) (value "MountingHole") (footprint "MountingHole:MountingHole_2.2mm_M2")
-    )
-    (path "/fc065b92-de59-4c29-93b4-0f722018f063/1ab5f143-cd2d-454a-b85a-745d6bcbefd9"
-      (reference "H6") (unit 1) (value "MountingHole") (footprint "MountingHole:MountingHole_2.2mm_M2")
-    )
-    (path "/fc065b92-de59-4c29-93b4-0f722018f063/597052a2-ccc6-450d-a467-b40f73c04c33"
-      (reference "H7") (unit 1) (value "MountingHole") (footprint "MountingHole:MountingHole_2.2mm_M2")
-    )
-    (path "/fc065b92-de59-4c29-93b4-0f722018f063/b79eb2df-c6d4-4428-b451-945a51eb4f71"
-      (reference "H8") (unit 1) (value "MountingHole") (footprint "MountingHole:MountingHole_2.2mm_M2")
-    )
-    (path "/0c7df807-3073-4929-bb80-e67459aef9d0/0e7162ec-2a3b-48b4-bfc6-544a081e3c69"
-      (reference "H9") (unit 1) (value "MountingHole") (footprint "MountingHole:MountingHole_2.2mm_M2")
-    )
-    (path "/0c7df807-3073-4929-bb80-e67459aef9d0/fc186107-614d-4fad-a412-e1ab324be828"
-      (reference "H10") (unit 1) (value "MountingHole") (footprint "MountingHole:MountingHole_2.2mm_M2")
-    )
-    (path "/0c7df807-3073-4929-bb80-e67459aef9d0/d89d2e45-e849-429a-a993-97c57a38406f"
-      (reference "H11") (unit 1) (value "MountingHole") (footprint "MountingHole:MountingHole_2.2mm_M2")
-    )
-    (path "/0c7df807-3073-4929-bb80-e67459aef9d0/e3ee739b-afee-4102-982c-9be831b76ee3"
-      (reference "H12") (unit 1) (value "MountingHole") (footprint "MountingHole:MountingHole_2.2mm_M2")
-    )
-    (path "/aeae0bd8-91e2-461e-89fa-f66aa100089e/0874bc0c-ee51-4de4-a724-fc1889d8781d"
-      (reference "H13") (unit 1) (value "MountingHole") (footprint "MountingHole:MountingHole_2.2mm_M2")
-    )
-    (path "/aeae0bd8-91e2-461e-89fa-f66aa100089e/dcd1d32e-6422-4d14-ba4a-4f91253a9c0f"
-      (reference "H14") (unit 1) (value "MountingHole") (footprint "MountingHole:MountingHole_2.2mm_M2")
-    )
-    (path "/aeae0bd8-91e2-461e-89fa-f66aa100089e/4d17ca8d-c20c-4f75-a277-8539f4896e82"
-      (reference "H15") (unit 1) (value "MountingHole") (footprint "MountingHole:MountingHole_2.2mm_M2")
-    )
-    (path "/aeae0bd8-91e2-461e-89fa-f66aa100089e/f86ae4a3-0890-4a5c-950c-ec42859cbec0"
-      (reference "H16") (unit 1) (value "MountingHole") (footprint "MountingHole:MountingHole_2.2mm_M2")
     )
     (path "/381ec3c9-e67f-421f-a889-e25a24188743"
@@
       (reference "TP2") (unit 1) (value "TestPoint_Harwin") (footprint "My Libraries:Harwin-S1751-46-Test-Point")
     )
-    (path "/2a737751-d85e-4f05-8aec-b659f83530c3/9d6f9a7d-51f4-4762-ae81-339c5995a8ca"
+    (path "/a4dae03d-0c29-490c-aab0-bcdda5d7deeb"
       (reference "TP3") (unit 1) (value "TestPoint_Harwin") (footprint "My Libraries:Harwin-S1751-46-Test-Point")
     )
@@
       (reference "TP11") (unit 1) (value "TestPoint_Harwin") (footprint "My Libraries:Harwin-S1751-46-Test-Point")
     )
-    (path "/fc065b92-de59-4c29-93b4-0f722018f063/0707396f-029d-4b28-b20e-006ae72e0a1b"
-      (reference "TP12") (unit 1) (value "TestPoint_Harwin") (footprint "My Libraries:Harwin-S1751-46-Test-Point")
-    )
     (path "/fc065b92-de59-4c29-93b4-0f722018f063/43215ec4-6e4b-4ce3-be6b-8af0514dd093"
       (reference "TP13") (unit 1) (value "TestPoint_Harwin") (footprint "My Libraries:Harwin-S1751-46-Test-Point")
@@
       (reference "TP20") (unit 1) (value "TestPoint_Harwin") (footprint "My Libraries:Harwin-S1751-46-Test-Point")
     )
-    (path "/0c7df807-3073-4929-bb80-e67459aef9d0/942dda87-e4ce-450a-8b1b-e525456b7d37"
-      (reference "TP21") (unit 1) (value "TestPoint_Harwin") (footprint "My Libraries:Harwin-S1751-46-Test-Point")
-    )
     (path "/0c7df807-3073-4929-bb80-e67459aef9d0/334b2057-7353-428e-9a61-41332810360f"
       (reference "TP22") (unit 1) (value "TestPoint_Harwin") (footprint "My Libraries:Harwin-S1751-46-Test-Point")
@@
       (reference "TP25") (unit 1) (value "TestPoint_Harwin") (footprint "My Libraries:Harwin-S1751-46-Test-Point")
     )
-    (path "/aeae0bd8-91e2-461e-89fa-f66aa100089e/f7e54589-ee92-4471-9d92-064a57749afe"
-      (reference "TP26") (unit 1) (value "TestPoint_Harwin") (footprint "My Libraries:Harwin-S1751-46-Test-Point")
-    )
     (path "/aeae0bd8-91e2-461e-89fa-f66aa100089e/f9fc8b9f-a8d8-4e68-be4b-36a54206d91b"

Commit message: pre-routing try 1
Parts:
- added JP2: 15V_byp, Jumper:SolderJumper-2_P1.3mm_Open_TrianglePad1.0x1.5mm, symbol Jumper:Jumper_2_Open
Connections:
- net 15v_Raw: now also JP2.1 (A)
- net Vin: now also JP2.2 (B)
- net mega_5v: now also J3.5 (Pin_5); no longer J3.7 (Pin_7)
- net stb_5v: now also J3.7 (Pin_7); no longer J3.5 (Pin_5)
Other:
- note added: "header for each supply solder jumper to bypass 15V"
Changed lines of the file:
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@@
   (no_connect (at 161.29 140.97))
   (no_connect (at 148.59 140.97))
-  (wire (pts (xy 119.38 96.52) (xy 119.38 135.89))
-    (stroke (width 0) (type default) (color 0 0 0 0))
-  )
   (wire (pts (xy 255.27 143.51) (xy 255.27 146.05))
     (stroke (width 0) (type default) (color 0 0 0 0))
@@
     (stroke (width 0) (type default) (color 0 0 0 0))
   )
+  (wire (pts (xy 114.3 96.52) (xy 114.3 138.43))
+    (stroke (width 0) (type default) (color 0 0 0 0))
+  )
   (wire (pts (xy 21.59 111.76) (xy 21.59 55.88))
     (stroke (width 0) (type default) (color 0 0 0 0))
@@
     (stroke (width 0) (type default) (color 0 0 0 0))
   )
-  (wire (pts (xy 119.38 135.89) (xy 148.59 135.89))
+  (wire (pts (xy 118.11 135.89) (xy 148.59 135.89))
     (stroke (width 0) (type default) (color 0 0 0 0))
   )
@@
     (stroke (width 0) (type default) (color 0 0 0 0))
   )
+  (wire (pts (xy 83.82 119.38) (xy 96.52 119.38))
+    (stroke (width 0) (type default) (color 0 0 0 0))
+  )
+  (wire (pts (xy 60.96 119.38) (xy 73.66 119.38))
+    (stroke (width 0) (type default) (color 0 0 0 0))
+  )
   (wire (pts (xy 63.5 130.81) (xy 72.39 130.81))
     (stroke (width 0) (type default) (color 0 0 0 0))
@@
     (stroke (width 0) (type default) (color 0 0 0 0))
   )
-  (wire (pts (xy 114.3 55.88) (xy 114.3 138.43))
-    (stroke (width 0) (type default) (color 0 0 0 0))
-  )
   (wire (pts (xy 127 101.6) (xy 127 133.35))
     (stroke (width 0) (type default) (color 0 0 0 0))
@@
     (stroke (width 0) (type default) (color 0 0 0 0))
   )
-  (wire (pts (xy 105.41 55.88) (xy 114.3 55.88))
+  (wire (pts (xy 105.41 55.88) (xy 118.11 55.88))
     (stroke (width 0) (type default) (color 0 0 0 0))
   )
@@
     (stroke (width 0) (type default) (color 0 0 0 0))
   )
+  (wire (pts (xy 118.11 55.88) (xy 118.11 135.89))
+    (stroke (width 0) (type default) (color 0 0 0 0))
+  )
   (wire (pts (xy 21.59 55.88) (xy 21.59 35.56))
     (stroke (width 0) (type default) (color 0 0 0 0))
@@
     (stroke (width 0) (type default) (color 0 0 0 0))
   )
-  (wire (pts (xy 63.5 96.52) (xy 119.38 96.52))
+  (wire (pts (xy 63.5 96.52) (xy 114.3 96.52))
     (stroke (width 0) (type default) (color 0 0 0 0))
   )
@@
   (wire (pts (xy 63.5 138.43) (xy 63.5 140.97))
     (stroke (width 0) (type default) (color 0 0 0 0))
+  )
+  (text "header for each supply\nsolder jumper to bypass 15V"
+    (at 104.14 26.67 0)
+    (effects (font (size 1.27 1.27)) (justify left bottom))
   )
   (label "Pos12_Out" (at 243.84 118.11 270)
     (effects (font (size 1.27 1.27)) (justify right bottom))
   )
+  (label "15v_Raw" (at 60.96 119.38 0)
+    (effects (font (size 1.27 1.27)) (justify left bottom))
+  )
   (label "Neg12_Out" (at 255.27 118.11 270)
     (effects (font (size 1.27 1.27)) (justify right bottom))
@@
     (effects (font (size 1.27 1.27)) (justify right bottom))
   )
-  (label "stb_5v" (at 147.32 135.89 180)
+  (label "stb_5v" (at 147.32 138.43 180)
+    (effects (font (size 1.27 1.27)) (justify right bottom))
+  )
+  (label "Vin" (at 96.52 119.38 180)
     (effects (font (size 1.27 1.27)) (justify right bottom))
   )
@@
     (effects (font (size 1.27 1.27)) (justify left bottom))
   )
-  (label "mega_5v" (at 147.186 138.43 180)
+  (label "mega_5v" (at 147.32 135.89 180)
     (effects (font (size 1.27 1.27)) (justify right bottom))
   )
@@
     (pin "2")
   )
+  (symbol (lib_id "Jumper:Jumper_2_Open") (at 78.74 119.38 0) (unit 1)
+    (in_bom yes) (on_board yes) (fields_autoplaced)
+    (property "Reference" "JP2" (id 0) (at 78.74 113.03 0))
+    (property "Value" "15V_byp" (id 1) (at 78.74 115.57 0))
+    (property "Footprint" "Jumper:SolderJumper-2_P1.3mm_Open_TrianglePad1.0x1.5mm" (id 2) (at 78.74 119.38 0)
+      (effects (font (size 1.27 1.27)) hide)
+    )
+    (property "Datasheet" "~" (id 3) (at 78.74 119.38 0)
+      (effects (font (size 1.27 1.27)) hide)
+    )
+    (pin "1")
+    (pin "2")
+  )
   (sheet (at 77.47 44.45) (size 27.94 25.4) (fields_autoplaced)
     (stroke (width 0.1524) (type solid) (color 0 0 0 0))
@@
       (reference "#PWR0118") (unit 1) (value "GND") (footprint "")
     )
+    (path "/2a737751-d85e-4f05-8aec-b659f83530c3/da5e3a38-f95a-4b3b-8980-9c323c38f68e"
+      (reference "#PWR0119") (unit 1) (value "GND") (footprint "")
+    )
     (path "/fc065b92-de59-4c29-93b4-0f722018f063/c35a082e-733e-4427-b04c-9802e85913c2"
       (reference "#PWR0120") (unit 1) (value "GND") (footprint "")
@@
     )
     (path "/2a737751-d85e-4f05-8aec-b659f83530c3/8ab5648e-985e-4a05-a058-8fe846c22de5"
-      (reference "C4") (unit 1) (value "100n") (footprint "Capacitor_SMD:C_0805_2012Metric")
+      (reference "C4") (unit 1) (value "100n") (footprint "Capacitor_SMD:C_0603_1608Metric")
     )
     (path "/2a737751-d85e-4f05-8aec-b659f83530c3/5a50c58b-952c-433f-afa1-8aa100bf3414"
@@
       (reference "C8") (unit 1) (value "470p") (footprint "Capacitor_SMD:C_0603_1608Metric")
     )
+    (path "/2a737751-d85e-4f05-8aec-b659f83530c3/55fa390e-747d-44a2-980f-28dca0a8a92f"
+      (reference "C9") (unit 1) (value "1u") (footprint "Capacitor_SMD:C_0805_2012Metric")
+    )
     (path "/fc065b92-de59-4c29-93b4-0f722018f063/c574b3be-f25a-4a58-9138-6a3766aa0952"
       (reference "C10") (unit 1) (value "10u") (footprint "Capacitor_SMD:C_0805_2012Metric")
@@
       (reference "JP1") (unit 1) (value "15V_Jmp") (footprint "Jumper:SolderJumper-2_P1.3mm_Open_TrianglePad1.0x1.5mm")
     )
+    (path "/f6551d38-e4fa-4b11-b3b5-b82f0db69be3"
+      (reference "JP2") (unit 1) (value "15V_byp") (footprint "Jumper:SolderJumper-2_P1.3mm_Open_TrianglePad1.0x1.5mm")
+    )
+    (path "/2a737751-d85e-4f05-8aec-b659f83530c3/cb629906-f5fc-4afc-8806-f8f3ec39b04c"
+      (reference "JP3") (unit 1) (value "neg_12_jmp") (footprint "Jumper:SolderJumper-2_P1.3mm_Open_TrianglePad1.0x1.5mm")
+    )
+    (path "/0c7df807-3073-4929-bb80-e67459aef9d0/c1b03037-b445-4091-ba05-e1412b30df60"
+      (reference "JP4") (unit 1) (value "mega_5v_jmp") (footprint "Jumper:SolderJumper-2_P1.3mm_Open_TrianglePad1.0x1.5mm")
+    )
+    (path "/aeae0bd8-91e2-461e-89fa-f66aa100089e/2c9c95fd-effd-47f0-9a8d-cb4301007e7e"
+      (reference "JP5") (unit 1) (value "stb_5v_jmp") (footprint "Jumper:SolderJumper-2_P1.3mm_Open_TrianglePad1.0x1.5mm")
+    )
     (path "/2a737751-d85e-4f05-8aec-b659f83530c3/4a24b938-7269-4636-98d1-7878c5d5806e"
       (reference "L1") (unit 1) (value "68u") (footprint "Inductor_SMD:L_Taiyo-Yuden_NR-80xx")
@@
     )
     (path "/2a737751-d85e-4f05-8aec-b659f83530c3/a902a587-b1c6-4ec1-ab6e-d046b860ddfe"
-      (reference "R1") (unit 1) (value "R") (footprint "Resistor_SMD:R_0805_2012Metric")
+      (reference "R1") (unit 1) (value "R") (footprint "Resistor_SMD:R_0402_1005Metric")
     )
     (path "/2a737751-d85e-4f05-8aec-b659f83530c3/da3d6292-ba43-40b5-921c-1d6babfe980d"
@@
       (reference "R3") (unit 1) (value "422k") (footprint "Resistor_SMD:R_0805_2012Metric")
     )
-    (path "/2a737751-d85e-4f05-8aec-b659f83530c3/e12ef5d2-ada9-4de8-9f6a-eca134421811"
-      (reference "R4") (unit 1) (value "0") (footprint "Resistor_SMD:R_0805_2012Metric")
-    )
     (path "/2a737751-d85e-4f05-8aec-b659f83530c3/746d76a2-1fb0-4806-8a95-90549d05b083"
       (reference "R5") (unit 1) (value "33k") (footprint "Resistor_SMD:R_0805_2012Metric")
     )
-    (path "/2a737751-d85e-4f05-8aec-b659f83530c3/339ea581-ce53-4d7c-a79b-af43280e2790"
-      (reference "R6") (unit 1) (value "1k") (footprint "Resistor_SMD:R_0805_2012Metric")
-    )
     (path "/c92524a7-c8a5-4c1e-a862-b184bdbc3f93"
       (reference "R7") (unit 1) (value "100") (footprint "Resistor_SMD:R_0805_2012Metric")
@@
       (reference "R25") (unit 1) (value "10k") (footprint "Resistor_SMD:R_0603_1608Metric")
     )
-    (path "/2a737751-d85e-4f05-8aec-b659f83530c3/af9d65c6-d176-4ffd-9005-1ee648989c77"
-      (reference "TP1") (unit 1) (value "TestPoint_Harwin") (footprint "My Libraries:Harwin-S1751-46-Test-Point")
-    )
-    (path "/2a737751-d85e-4f05-8aec-b659f83530c3/e312b235-fa9d-4146-a238-9cc6d5599ffa"
-      (reference "TP2") (unit 1) (value "TestPoint_Harwin") (footprint "My Libraries:Harwin-S1751-46-Test-Point")
-    )
     (path "/a4dae03d-0c29-490c-aab0-bcdda5d7deeb"
       (reference "TP3") (unit 1) (value "TestPoint_Harwin") (footprint "My Libraries:Harwin-S1751-46-Test-Point")
     )
-    (path "/2a737751-d85e-4f05-8aec-b659f83530c3/7761274e-b4ac-41b9-939c-99d416e203db"
-      (reference "TP4") (unit 1) (value "TestPoint_Harwin") (footprint "My Libraries:Harwin-S1751-46-Test-Point")
-    )
     (path "/2a737751-d85e-4f05-8aec-b659f83530c3/ce42903e-1fd1-436b-8ae3-9c2a4886379e"
-      (reference "TP5") (unit 1) (value "TestPoint_Harwin") (footprint "My Libraries:Harwin-S1751-46-Test-Point")
+      (reference "TP5") (unit 1) (value "TestPoint_Harwin") (footprint "TestPoint:TestPoint_Pad_1.0x1.0mm")
     )
     (path "/2a737751-d85e-4f05-8aec-b659f83530c3/107fb3c5-9f1e-428d-b18d-cb090cb19861"
-      (reference "TP6") (unit 1) (value "TestPoint_Harwin") (footprint "My Libraries:Harwin-S1751-46-Test-Point")
+      (reference "TP6") (unit 1) (value "TestPoint_Harwin") (footprint "TestPoint:TestPoint_Pad_1.0x1.0mm")
     )
     (path "/2a737751-d85e-4f05-8aec-b659f83530c3/76c57c21-eeda-4bfc-91bf-cf08d7b5d793"
@@
     )
     (path "/2a737751-d85e-4f05-8aec-b659f83530c3/3d812d77-839b-4dbe-a58c-f3b7ccfebe96"
-      (reference "TP8") (unit 1) (value "TestPoint_Harwin") (footprint "My Libraries:Harwin-S1751-46-Test-Point")
+      (reference "TP8") (unit 1) (value "TestPoint_Harwin") (footprint "TestPoint:TestPoint_Pad_1.0x1.0mm")
     )
     (path "/2a737751-d85e-4f05-8aec-b659f83530c3/4174bae9-405e-4ccd-b0d5-bcd07e58bba4"
