File: kicad files/gd power supply board pcb/gd power supply board pcb.kicad_sch (KiCad schematic)
At the start: 25 parts, among them J1 15V_IN, J2 15V_IN, J3 Edge Connector, Q1 FDS9435A

Commit message: 0 unrouted - drc pass - need to clean silks
Connections:
- net Analog_En: now also J3.12 (Pin_12); no longer J3.11 (Pin_11)
- net Mega_En: now also J3.11 (Pin_11); no longer J3.12 (Pin_12)
- net mega_5v: now also J3.7 (Pin_7); no longer J3.5 (Pin_5)
- net stb_5v: now also J3.5 (Pin_5); no longer J3.7 (Pin_7)
Changed lines of the file:
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@@
     (stroke (width 0) (type default) (color 0 0 0 0))
   )
-  (wire (pts (xy 123.19 60.96) (xy 123.19 143.51))
+  (wire (pts (xy 123.19 60.96) (xy 123.19 152.4))
     (stroke (width 0) (type default) (color 0 0 0 0))
   )
@@
     (stroke (width 0) (type default) (color 0 0 0 0))
   )
-  (wire (pts (xy 114.3 96.52) (xy 114.3 138.43))
+  (wire (pts (xy 114.3 96.52) (xy 114.3 135.89))
     (stroke (width 0) (type default) (color 0 0 0 0))
   )
@@
     (stroke (width 0) (type default) (color 0 0 0 0))
   )
-  (wire (pts (xy 118.11 135.89) (xy 148.59 135.89))
-    (stroke (width 0) (type default) (color 0 0 0 0))
-  )
   (wire (pts (xy 215.9 62.23) (xy 215.9 40.64))
     (stroke (width 0) (type default) (color 0 0 0 0))
@@
     (stroke (width 0) (type default) (color 0 0 0 0))
   )
-  (wire (pts (xy 114.3 138.43) (xy 148.59 138.43))
+  (wire (pts (xy 110.49 146.05) (xy 139.7 146.05))
     (stroke (width 0) (type default) (color 0 0 0 0))
   )
@@
     (stroke (width 0) (type default) (color 0 0 0 0))
   )
-  (wire (pts (xy 148.59 143.51) (xy 123.19 143.51))
-    (stroke (width 0) (type default) (color 0 0 0 0))
-  )
   (wire (pts (xy 255.27 118.11) (xy 255.27 130.81))
     (stroke (width 0) (type default) (color 0 0 0 0))
@@
     (stroke (width 0) (type default) (color 0 0 0 0))
   )
+  (wire (pts (xy 123.19 152.4) (xy 173.99 152.4))
+    (stroke (width 0) (type default) (color 0 0 0 0))
+  )
   (wire (pts (xy 195.58 143.51) (xy 195.58 146.05))
     (stroke (width 0) (type default) (color 0 0 0 0))
@@
     (stroke (width 0) (type default) (color 0 0 0 0))
   )
+  (wire (pts (xy 139.7 143.51) (xy 148.59 143.51))
+    (stroke (width 0) (type default) (color 0 0 0 0))
+  )
+  (wire (pts (xy 118.11 138.43) (xy 148.59 138.43))
+    (stroke (width 0) (type default) (color 0 0 0 0))
+  )
   (wire (pts (xy 219.71 57.15) (xy 219.71 35.56))
     (stroke (width 0) (type default) (color 0 0 0 0))
@@
     (stroke (width 0) (type default) (color 0 0 0 0))
   )
+  (wire (pts (xy 139.7 143.51) (xy 139.7 146.05))
+    (stroke (width 0) (type default) (color 0 0 0 0))
+  )
   (wire (pts (xy 30.48 129.54) (xy 27.94 129.54))
     (stroke (width 0) (type default) (color 0 0 0 0))
@@
     (stroke (width 0) (type default) (color 0 0 0 0))
   )
-  (wire (pts (xy 110.49 146.05) (xy 173.99 146.05))
-    (stroke (width 0) (type default) (color 0 0 0 0))
-  )
   (wire (pts (xy 219.71 35.56) (xy 128.27 35.56))
     (stroke (width 0) (type default) (color 0 0 0 0))
@@
     (stroke (width 0) (type default) (color 0 0 0 0))
   )
-  (wire (pts (xy 118.11 55.88) (xy 118.11 135.89))
+  (wire (pts (xy 118.11 55.88) (xy 118.11 138.43))
     (stroke (width 0) (type default) (color 0 0 0 0))
   )
@@
     (stroke (width 0) (type default) (color 0 0 0 0))
   )
+  (wire (pts (xy 148.59 135.89) (xy 114.3 135.89))
+    (stroke (width 0) (type default) (color 0 0 0 0))
+  )
   (wire (pts (xy 105.41 130.81) (xy 105.41 111.76))
     (stroke (width 0) (type default) (color 0 0 0 0))
@@
     (stroke (width 0) (type default) (color 0 0 0 0))
   )
-  (wire (pts (xy 173.99 143.51) (xy 173.99 146.05))
+  (wire (pts (xy 173.99 143.51) (xy 173.99 152.4))
     (stroke (width 0) (type default) (color 0 0 0 0))
   )
@@
     (effects (font (size 1.27 1.27)) (justify right bottom))
   )
-  (label "stb_5v" (at 147.32 138.43 180)
-    (effects (font (size 1.27 1.27)) (justify right bottom))
+  (label "stb_5v" (at 138.43 135.89 0)
+    (effects (font (size 1.27 1.27)) (justify left bottom))
   )
   (label "Vin" (at 96.52 119.38 180)
@@
     (effects (font (size 1.27 1.27)) (justify left bottom))
   )
-  (label "Mega_En" (at 173.99 143.51 180)
-    (effects (font (size 1.27 1.27)) (justify right bottom))
+  (label "Mega_En" (at 139.7 143.51 0)
+    (effects (font (size 1.27 1.27)) (justify left bottom))
   )
   (label "Pos12_Out" (at 137.16 133.35 0)
     (effects (font (size 1.27 1.27)) (justify left bottom))
   )
-  (label "mega_5v" (at 147.32 135.89 180)
-    (effects (font (size 1.27 1.27)) (justify right bottom))
+  (label "mega_5v" (at 138.43 138.43 0)
+    (effects (font (size 1.27 1.27)) (justify left bottom))
   )
   (label "15v_Raw" (at 20.32 124.46 0)
     (effects (font (size 1.27 1.27)) (justify left bottom))
   )
-  (label "Analog_En" (at 137.16 143.51 0)
-    (effects (font (size 1.27 1.27)) (justify left bottom))
+  (label "Analog_En" (at 172.72 143.51 180)
+    (effects (font (size 1.27 1.27)) (justify right bottom))
   )
   (label "mega_5v" (at 217.17 118.11 270)
