File: kicad files/gd power supply board pcb/proto socket adapter/proto socket adapter.kicad_sch (KiCad schematic)
At the start: 6 parts, among them J1 Right Angle, J2 Rev2 Header, J3 RP2040 Header, J4 Straight

Commit message: sub rev1 to fab
Parts:
- removed J4: Straight, My Libraries:Sullins-EBC06DCWN-Edge Socket 12 pos (6x2), symbol Connector_Generic:Conn_02x06_Odd_Even
- removed J?: RP2040 Header, Connector_PinSocket_2.54mm:PinSocket_2x03_P2.54mm_Vertical, symbol Connector_Generic:Conn_02x03_Odd_Even
- removed J?: Rev2 Header, Connector_PinSocket_2.54mm:PinSocket_2x04_P2.54mm_Vertical, symbol Connector_Generic:Conn_02x04_Odd_Even
- added D1: -12v, LED_SMD:LED_0805_2012Metric, symbol My Library:D_1206
- added D2: +12v, LED_SMD:LED_0805_2012Metric, symbol My Library:D_1206
- added D3: Mega, LED_SMD:LED_0805_2012Metric, symbol My Library:D_1206
- added D4: Stby, LED_SMD:LED_0805_2012Metric, symbol My Library:D_1206
- added H1, H2: MountingHole, MountingHole:MountingHole_2.2mm_M2, symbol Mechanical:MountingHole
- added R1, R2, R3, R4: 1K, Resistor_SMD:R_0805_2012Metric, symbol My Library:R_0805
Connections:
- net Analog_En: now also J3.1 (Pin_1); no longer J3.6 (Pin_6)
- net GND: now also J3.3 (Pin_3), J3.4 (Pin_4), D2.1 (K), D3.1 (K), D4.1 (K), R1.1; no longer J3.1 (Pin_1), J3.2 (Pin_2)
- net Mega_En: now also J3.2 (Pin_2); no longer J3.5 (Pin_5)
- net Neg12_Out: now also D1.1 (K)
- net Pos12_Out: now also R2.1
- net mega_5v: now also R4.1
- net stb_5v: now also J3.5 (Pin_5), J3.6 (Pin_6), R3.1; no longer J3.3 (Pin_3), J3.4 (Pin_4)
- new net: D2.2 (A), R2.2
- new net: D4.2 (A), R3.2
- new net: D3.2 (A), R4.2
- new net: D1.2 (A), R1.2
- no-connect marks 4 -> 2
