File: kicad files/gd io proto pcb/gd io proto pcb.kicad_sch (KiCad schematic)
At the start: 36 parts, among them J1 Pwr, J10 DEV LA, J11 Annunciate, J12 Apple_II_Slot, J13 Slot Maker, J14 Slot Maker LA, J15 Slot-Only Sigs, J16 IO Selector, J17 -5V, J18 IOSEL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

Commit message: resolved ERC errors, like fixing en245...wth?
Connections:
- net EN245 is gone; now on net ~{EN245}: U2.19 (G)
Other:
- moved on the sheet: J1

Commit message: resolves #57. now there is a 2-pin header for dev select (and a pin to probe with logic analyzer.) also fixed an issue with the 245 enable signal (whoops.)
Parts:
- added J19: DEVx, Connector_PinHeader_2.54mm:PinHeader_1x02_P2.54mm_Vertical, symbol Connector_Generic:Conn_01x02
- U2: value 74HCT245-CHECK FOOTPRINT -> 74HCT245
Connections:
- net ~{DEV1}: no longer J12.41
- new net ~{DEVx}: J12.41, J19.1 (Pin_1), J19.2 (Pin_2)
Other:
- moved on the sheet: C1, C3, C4, C6, C7, D2, D4, D5, D7, J18, R2, R4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

Commit message: fixed sbus signals (#18)
Connections:
- net SBUS0: now also U1.11 (S0); no longer U1.6 (S5)
- net SBUS1: now also U1.10 (S1); no longer U1.7 (S4)
- net SBUS2: now also U1.9 (S2); no longer U1.8 (S3)
- net SBUS3: now also U1.8 (S3); no longer U1.9 (S2)
- net SBUS4: now also U1.7 (S4); no longer U1.10 (S1)
- net SBUS5: now also U1.6 (S5); no longer U1.11 (S0)
Changed lines of the file:
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@@
     (effects (font (size 1.27 1.27)) (justify left bottom))
   )
-  (label "SBUS4" (at 57.15 86.36 0) (fields_autoplaced)
+  (label "SBUS4" (at 57.15 78.74 0) (fields_autoplaced)
     (effects (font (size 1.27 1.27)) (justify left bottom))
   )
@@
     (effects (font (size 1.27 1.27)) (justify right bottom))
   )
-  (label "SBUS0" (at 57.15 76.2 0) (fields_autoplaced)
+  (label "SBUS0" (at 57.15 88.9 0) (fields_autoplaced)
     (effects (font (size 1.27 1.27)) (justify left bottom))
   )
@@
     (effects (font (size 1.27 1.27)) (justify left bottom))
   )
-  (label "SBUS3" (at 57.15 83.82 0) (fields_autoplaced)
+  (label "SBUS3" (at 57.15 81.28 0) (fields_autoplaced)
     (effects (font (size 1.27 1.27)) (justify left bottom))
   )
@@
     (effects (font (size 1.27 1.27)) (justify left bottom))
   )
-  (label "SBUS5" (at 57.15 88.9 0) (fields_autoplaced)
+  (label "SBUS5" (at 57.15 76.2 0) (fields_autoplaced)
     (effects (font (size 1.27 1.27)) (justify left bottom))
   )
@@
     (effects (font (size 1.27 1.27)) (justify right bottom))
   )
-  (label "SBUS2" (at 57.15 81.28 0) (fields_autoplaced)
+  (label "SBUS2" (at 57.15 83.82 0) (fields_autoplaced)
     (effects (font (size 1.27 1.27)) (justify left bottom))
   )
@@
     (effects (font (size 1.27 1.27)) (justify right bottom))
   )
-  (label "SBUS1" (at 57.15 78.74 0) (fields_autoplaced)
-    (effects (font (size 1.27 1.27)) (justify left bottom))
-  )
+  (label "SBUS1" (at 57.15 86.36 0) (fields_autoplaced)
+    (effects (font (size 1.27 1.27)) (justify left bottom))
+  )
