File: kicad files/gd io proto pcb/gd iwm rom card pcb/gd iwm rom card pcb.kicad_sch (KiCad schematic)
At the start: 12 parts, among them J1 Apple_II_Slot, U1 27C512, U2 74HCT245-CHECK FOOTPRINT

Commit message: primary components in schematic
Parts:
- added C2: 1uF, Capacitor_SMD:C_0805_2012Metric, symbol Device:C_Small
- added U3: 74HC245, Package_SO:SOIC-20W_7.5x12.8mm_P1.27mm, symbol gd-io-proto-pcb-rescue:74HCT245-Apple_IIgs_Symbols
- added U4: ~, symbol My Library:GAL20V8
- added U5: 74LS21, Package_SO:SO-14_3.9x8.65mm_P1.27mm, symbol 74xx:74LS21
- U2: value 74HCT245-CHECK FOOTPRINT -> 74HC245; footprint Package_SO:SO-20_12.8x7.5mm_P1.27mm -> Package_SO:SOIC-20W_7.5x12.8mm_P1.27mm
Connections:
- net +5V: now also C2.1, U4.24 (VCC)
- net GND: now also U2.10 (GND), C2.2, U3.10 (GND), U4.12 (GND), U4.13 (I13/~{OE})
- net ~{IOSEL}: now also U4.8 (I8)
- net ~{RESET}: now also U4.11 (I11)
- new net A0: U4.5 (I5)
- new net A1: U4.4 (I4)
- new net A10: U5.12
- new net A2: U4.3 (I3)
- new net A3: U4.2 (i2)
- new net A4: U5.1
- new net A5: U5.2
- new net A6: U5.4
- new net A7: U5.5
- new net A8: U5.9
- new net A9: U5.10
- new net D0: U4.6 (I6)
- new net FF1: U4.23 (I23), U5.6
- new net FF2: U4.22 (IO22), U5.8
- new net PHI1: U4.1 (I1)
- new net PI_EN: U4.15 (IO15)
- new net PI_OE: U4.16 (IO16)
- new net RAM_A12: U4.19 (IO19)
- new net RAM_EN: U4.17 (IO17)
- new net R/~{W}: U4.10 (I10)
- new net ~{DEVSEL}: U4.7 (I7)
- new net ~{INHIBIT}: U4.14 (I14)
- new net ~{IOSTROBE}: U4.9 (I9)
- new net ~{RAM_OE}: U4.18 (IO18)
- no-connect marks 1 -> 3
Other:
- company: (none) -> baldengineer.com
- title: (none) -> IWM ROM Card Proto
- moved on the sheet: C1, U1

Commit message: r1 layout done, needs review
Parts:
- removed J1: Apple_II_Slot, My Libraries:Amp_2358256-4_50pos_right_angle_card, symbol gd-io-proto-pcb-rescue:Apple_II_Slot-Apple_IIgs_Symbols
- added C3, C4, C5: 1uF, Capacitor_SMD:C_0805_2012Metric, symbol Device:C_Small
- added C6: 47u, Capacitor_THT:CP_Radial_D5.0mm_P2.50mm, symbol Device:C_Polarized_Small
- added J1: CARD EDGE, My Libraries:AppleII_Bus, symbol Connector_Generic:Conn_02x25_Counter_Clockwise
- added J2: HEADER BLOCK, My Libraries:PinSocket_2x25_P2.54mm_Vertical_CCW_Mirrored_NoSilk, symbol Connector_Generic:Conn_02x25_Counter_Clockwise
- added JP1: PH, Jumper:SolderJumper-2_P1.3mm_Bridged_RoundedPad1.0x1.5mm, symbol Jumper:SolderJumper_2_Bridged
- added JP2, JP3, JP4, JP5: SolderJumper_3_Bridged12, Jumper:SolderJumper-3_P1.3mm_Bridged12_RoundedPad1.0x1.5mm_NumberLabels, symbol Jumper:SolderJumper_3_Bridged12
- added TP1, TP4, TP5, TP6, TP7: PH0, TestPoint:TestPoint_Pad_1.0x1.0mm, symbol Connector:TestPoint_Small
- added TP2: IO21, TestPoint:TestPoint_Pad_1.0x1.0mm, symbol Connector:TestPoint_Small
- added TP3: IO20, TestPoint:TestPoint_Pad_1.0x1.0mm, symbol Connector:TestPoint_Small
- added unit 3 of U5
- R1, R2, R3, R4: symbol gd-io-proto-pcb-rescue:R_0805-My_Library -> My Library:R_0805
- U2, U3: symbol gd-io-proto-pcb-rescue:74HCT245-Apple_IIgs_Symbols -> My Library:74HCT245_1
- U4: value ~ -> GAL20V8; footprint (none) -> Package_DIP:DIP-24_W7.62mm_Socket_LongPads
Connections:
- net MD0 is gone; now on net D0: U1.11 (D0)
- net ~{INHIBIT} is gone; now on net ~{INH}: U4.14 (I14)
- net ~{IOSTROBE} is gone; now on net ~{IOSTRB}: U4.9 (I9)
- net ~{ROMEN} is gone; now on net ~{ROM_OE}: U1.22 (~{OE})
- net +12V: now also J1.50 (Pin_50), J2.50 (Pin_50)
- net +5V: now also U2.1 (DIR), U2.20 (+V), U3.1 (DIR), U3.20 (+V), C3.1, C4.1, C5.1, C6.1, J1.25 (Pin_25), J2.25 (Pin_25), U5.14 (VCC)
- net -12V: now also J1.33 (Pin_33), J2.33 (Pin_33)
- net -5V: now also J1.34 (Pin_34), J2.34 (Pin_34)
- net A0: now also U2.2 (A1), J1.2 (Pin_2), J2.2 (Pin_2)
- net A1: now also U2.3 (A2), J1.3 (Pin_3), J2.3 (Pin_3)
- net A10: now also U3.4 (A3), U5.13, J1.12 (Pin_12), J2.12 (Pin_12)
- net A2: now also U2.4 (A3), J1.4 (Pin_4), J2.4 (Pin_4)
- net A3: now also U2.5 (A4), J1.5 (Pin_5), J2.5 (Pin_5)
- net A4: now also U2.6 (A5), J1.6 (Pin_6), J2.6 (Pin_6)
- net A5: now also U2.7 (A6), J1.7 (Pin_7), J2.7 (Pin_7)
- net A6: now also U2.8 (A7), J1.8 (Pin_8), J2.8 (Pin_8)
- net A7: now also U2.9 (A8), J1.9 (Pin_9), J2.9 (Pin_9)
- net A8: now also U3.2 (A1), J1.10 (Pin_10), J2.10 (Pin_10)
- net A9: now also U3.3 (A2), J1.11 (Pin_11), J2.11 (Pin_11)
- net BA0: now also U2.18 (B1)
- net BA1: now also U2.17 (B2)
- net BA10: now also U3.16 (B3)
- net BA11: now also U3.15 (B4)
- net BA12: now also U3.14 (B5), JP2.3 (B); no longer U1.2 (A12)
- net BA13: now also U3.13 (B6), JP3.3 (B); no longer U1.26 (A13)
- net BA14: now also U3.12 (B7), JP4.3 (B)
- net BA15: now also U3.11 (B8), JP5.3 (B)
- net BA2: now also U2.16 (B3)
- net BA3: now also U2.15 (B4)
- net BA4: now also U2.14 (B5)
- net BA5: now also U2.13 (B6)
- net BA6: now also U2.12 (B7)
- net BA7: now also U2.11 (B8)
- net BA8: now also U3.18 (B1)
- net BA9: now also U3.17 (B2)
- net D0: now also J1.49 (Pin_49), J2.49 (Pin_49)
- net GND: now also U2.19 (G), U3.19 (G), C3.2, C4.2, C5.2, C6.2, J1.26 (Pin_26), J2.26 (Pin_26), JP2.2 (C), JP3.2 (C), JP4.2 (C), JP5.2 (C), U5.7 (GND); no longer U1.1 (A15), U1.27 (A14)
- net PHI1: now also J1.38 (Pin_38), J2.38 (Pin_38), JP1.1 (A); no longer U4.1 (I1)
- net PI_EN: now also TP7.1
- net PI_OE: now also TP6.1
- net R/~{W}: now also J1.18 (Pin_18), J2.18 (Pin_18)
- net ~{DEVSEL}: now also J1.41 (Pin_41), J2.41 (Pin_41)
- net ~{DMA}: now also J1.22 (Pin_22), J2.22 (Pin_22)
- net ~{INH}: now also J1.32 (Pin_32), J2.32 (Pin_32)
- net ~{IOSEL}: now also J1.1 (Pin_1), J2.1 (Pin_1)
- net ~{IOSTRB}: now also J1.20 (Pin_20), J2.20 (Pin_20)
- net ~{IRQ}: now also J1.30 (Pin_30), J2.30 (Pin_30)
- net ~{NMI}: now also J1.29 (Pin_29), J2.29 (Pin_29)
- net ~{RESET}: now also J1.31 (Pin_31), J2.31 (Pin_31)
- net RAMEXEC: now reaches U4.20 (IO20)
- net RAMEXEC: now also TP3.1
- net C800_EXT: now reaches U4.21 (IO21)
- net C800_EXT: now also TP2.1
- net A11: now reaches U3.5 (A4)
- net A11: now also J1.13 (Pin_13), J2.13 (Pin_13)
- net A12: now reaches U3.6 (A5)
- net A12: now also J1.14 (Pin_14), J2.14 (Pin_14)
- net A13: now reaches U3.7 (A6)
- net A13: now also J1.15 (Pin_15), J2.15 (Pin_15)
- net A14: now reaches U3.8 (A7)
- net A14: now also J1.16 (Pin_16), J2.16 (Pin_16)
- net A15: now reaches U3.9 (A8)
- net A15: now also J1.17 (Pin_17), J2.17 (Pin_17)
- net MD1 renamed D1
- net D1: now also J1.48 (Pin_48), J2.48 (Pin_48)
- net MD2 renamed D2
- net D2: now also J1.47 (Pin_47), J2.47 (Pin_47)
- net MD3 renamed D3
- net D3: now also J1.46 (Pin_46), J2.46 (Pin_46)
- net MD4 renamed D4
- net D4: now also J1.45 (Pin_45), J2.45 (Pin_45)
- net MD5 renamed D5
- net D5: now also J1.44 (Pin_44), J2.44 (Pin_44)
- net MD6 renamed D6
- net D6: now also J1.43 (Pin_43), J2.43 (Pin_43)
- net MD7 renamed D7
- net D7: now also J1.42 (Pin_42), J2.42 (Pin_42)
- net RAM_A12 renamed ROM_A12
- net ROM_A12: now also TP4.1
- net RAM_EN renamed ROM_EN
- net ROM_EN: now also TP5.1
- net ~{RAM_OE} renamed ~{ROM_OE}
- new net: JP1.2 (B), U4.1 (I1)
- new net 7M: J1.36 (Pin_36), J2.36 (Pin_36)
- new net BBA12: JP2.1 (A), U1.2 (A12)
- new net BBA13: JP3.1 (A), U1.26 (A13)
- new net BBA14: JP4.1 (A), U1.27 (A14)
- new net BBA15: JP5.1 (A), U1.1 (A15)
- new net COLORREF: J1.35 (Pin_35), J2.35 (Pin_35)
- new net DMAIN: J1.27 (Pin_27), J2.27 (Pin_27)
- new net DMAOUT: J1.24 (Pin_24), J2.24 (Pin_24)
- new net INTIN: J1.28 (Pin_28), J2.28 (Pin_28)
- new net INTOUT: J1.23 (Pin_23), J2.23 (Pin_23)
- new net PHI0: J1.40 (Pin_40), J2.40 (Pin_40), TP1.1
- new net Q3: J1.37 (Pin_37), J2.37 (Pin_37)
- new net RDY: J1.21 (Pin_21), J2.21 (Pin_21)
- new net SYNC: J1.19 (Pin_19), J2.19 (Pin_19)
- new net USER1: J1.39 (Pin_39), J2.39 (Pin_39)
- no-connect marks 3 -> 0
Other:
- moved on the sheet: C1, C2, U1, U2, U3, U4, U5A, U5B
