File: kicad files/gd iwm rom card pcb/gd iwm rom card pcb.kicad_sch (KiCad schematic)
At the start: 33 parts, among them J1 CARD EDGE, J2 HEADER BLOCK, U1 27C512, U2 74HC245, U3 74HC245, U4 GAL20V8, U5 74LS21

Commit message: added notes
Other:
- note added: "CFFF 0111 xxx xxxx xxxx 1111 1100 0000 0000 5432 1098 7654 3210 ---- ---- ---- ---- 1100 1111 1111 1111 C7Fx - CFFx"
Changed lines of the file:
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@@
     (stroke (width 0) (type default))
+  )
+  (text "CFFF\n\n     0111\n      xxx xxxx xxxx\n1111 1100 0000 0000\n5432 1098 7654 3210\n---- ---- ---- ----\n1100 1111 1111 1111\n\n\nC7Fx - CFFx"
+    (at 298.45 92.075 0)
+    (effects (font (size 1.27 1.27)) (justify left bottom))
   )
   (label "FF1" (at 139.7 85.725 0) (fields_autoplaced)
