File: kicad files/gd rev3b/Audio.kicad_sch (KiCad schematic)
At the start: 18 parts, among them J19 SPKR, J20 Ears, Q2 BC817, U26 MCP4541T, U27 LM4875

Commit message: Schematic changes for #52, #50, #70, #51, #61, #69, #71
Connections:
- net at Q2.3 (C): now also R48.2; no longer R48.1
- net at D2.1 (K): now also R48.1; no longer R48.2
- net +5V renamed +5V_2040
Other:
- note added: "Q: Are we scaling the audio on demo board? A: I still don't know. Need to see what I did on R3 pcb."
- note removed: "Are we scaling the audio on demo board?"
- moved on the sheet: J20, R48
