File: kicad files/gd rev3b/power.kicad_sch (KiCad schematic)
At the start: 24 parts, among them J12 Right Angle, J15 PS Aux, J16 PS Control

Commit message: Schematic changes for #52, #50, #70, #51, #61, #69, #71
Parts:
- R27, R28, R29, R30: value 1K -> 4k7
Changed lines of the file:
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@@
+    (stroke (width 0) (type default))
+  )
+  (wire (pts (xy 137.795 163.195) (xy 137.795 161.925))
     (stroke (width 0) (type default))
   )
@@
   )
   (wire (pts (xy 180.34 87.63) (xy 184.15 87.63))
+    (stroke (width 0) (type default))
+  )
+  (wire (pts (xy 137.795 161.925) (xy 133.985 161.925))
     (stroke (width 0) (type default))
   )
@@
   (label "Analog_Pwr" (at 153.67 96.52 180) (fields_autoplaced)
     (effects (font (size 1.27 1.27)) (justify right bottom))
+  )
+  (label "GND" (at 133.985 161.925 0) (fields_autoplaced)
+    (effects (font (size 1.27 1.27)) (justify left bottom))
   )
   (label "stb_5v" (at 116.84 118.11 0) (fields_autoplaced)
@@
   (symbol (lib_id "Mega IIe Rev3 Symbols:R_0805") (at 64.77 133.35 0) (unit 1)
     (in_bom yes) (on_board yes) (dnp no) (fields_autoplaced)
-    (property "Reference" "R28" (at 67.31 132.0799 0)
-      (effects (font (size 1.27 1.27)) (justify left))
-    )
-    (property "Value" "1K" (at 67.31 134.6199 0)
+    (property "Reference" "R28" (at 67.31 132.08 0)
+      (effects (font (size 1.27 1.27)) (justify left))
+    )
+    (property "Value" "4k7" (at 67.31 134.62 0)
       (effects (font (size 1.27 1.27)) (justify left))
     )
@@
   (symbol (lib_id "Mega IIe Rev3 Symbols:R_0805") (at 90.17 133.35 0) (unit 1)
     (in_bom yes) (on_board yes) (dnp no) (fields_autoplaced)
-    (property "Reference" "R30" (at 92.71 132.0799 0)
-      (effects (font (size 1.27 1.27)) (justify left))
-    )
-    (property "Value" "1K" (at 92.71 134.6199 0)
+    (property "Reference" "R30" (at 92.71 132.08 0)
+      (effects (font (size 1.27 1.27)) (justify left))
+    )
+    (property "Value" "4k7" (at 92.71 134.62 0)
       (effects (font (size 1.27 1.27)) (justify left))
     )
@@
   )
   (symbol (lib_id "Mega IIe Rev3 Symbols:D_1206") (at 54.61 132.08 270) (unit 1)
-    (in_bom yes) (on_board yes) (dnp no) (fields_autoplaced)
+    (in_bom yes) (on_board yes) (dnp no)
     (property "Reference" "D4" (at 57.15 130.8099 90)
       (effects (font (size 1.27 1.27)) (justify left))
     )
-    (property "Value" "-12v" (at 57.15 133.3499 90)
+    (property "Value" "-12v" (at 55.88 132.715 90)
       (effects (font (size 1.27 1.27)) (justify left))
     )
@@
   (symbol (lib_id "Mega IIe Rev3 Symbols:R_0805") (at 54.61 138.43 180) (unit 1)
     (in_bom yes) (on_board yes) (dnp no) (fields_autoplaced)
-    (property "Reference" "R27" (at 52.07 139.7001 0)
-      (effects (font (size 1.27 1.27)) (justify left))
-    )
-    (property "Value" "1K" (at 52.07 137.1601 0)
-      (effects (font (size 1.27 1.27)) (justify left))
+    (property "Reference" "R27" (at 57.15 137.16 0)
+      (effects (font (size 1.27 1.27)) (justify right))
+    )
+    (property "Value" "4k7" (at 57.15 139.7 0)
+      (effects (font (size 1.27 1.27)) (justify right))
     )
     (property "Footprint" "Resistor_SMD:R_0805_2012Metric" (at 54.61 138.43 0)
@@
   (symbol (lib_id "Mega IIe Rev3 Symbols:R_0805") (at 77.47 133.35 0) (unit 1)
     (in_bom yes) (on_board yes) (dnp no) (fields_autoplaced)
-    (property "Reference" "R29" (at 80.01 132.0799 0)
-      (effects (font (size 1.27 1.27)) (justify left))
-    )
-    (property "Value" "1K" (at 80.01 134.6199 0)
+    (property "Reference" "R29" (at 80.01 132.08 0)
+      (effects (font (size 1.27 1.27)) (justify left))
+    )
+    (property "Value" "4k7" (at 80.01 134.62 0)
       (effects (font (size 1.27 1.27)) (justify left))
     )
@@
         )
       )
+    )
+  )
+  (symbol (lib_id "power:GND") (at 137.795 163.195 0) (unit 1)
+    (in_bom yes) (on_board yes) (dnp no)
+    (property "Reference" "#PWR0189" (at 137.795 169.545 0)
+      (effects (font (size 1.27 1.27)) hide)
+    )
+    (property "Value" "GND" (at 137.922 167.5892 0)
+      (effects (font (size 1.27 1.27)))
+    )
+    (property "Footprint" "" (at 137.795 163.195 0)
+      (effects (font (size 1.27 1.27)) hide)
+    )
+    (property "Datasheet" "" (at 137.795 163.195 0)
+      (effects (font (size 1.27 1.27)) hide)
+    )
+    (pin "1")
+    (instances
+      (project "gd rev3b"
+        (path "/e63e39d7-6ac0-4ffd-8aa3-1841a4541b55/a9c8f5ac-a28a-4770-a319-78cb5bb789be"
+          (reference "#PWR0189") (unit 1)
+        )
+        (path "/e63e39d7-6ac0-4ffd-8aa3-1841a4541b55/c78c3992-30f5-49be-b188-a14fa5a1512a"
+          (reference "#PWR019") (unit 1)
+        )
+      )
