File: kicad files/gd rev3b/rp2040-keyboard.kicad_sch (KiCad schematic)
At the start: 60 parts, among them J13 SWD, J14 USB_A, J21 KBD Serial, J24 KBD_L_HDR, Q10 BC817, Q3 BC817, SW4 KBD RESET, SW5 KBD Boot Sel, U14 RP2040, U15 MIC5504-3.3YM5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

Commit message: Schematic changes for #52, #50, #70, #51, #61, #69, #71
Parts:
- added D26, D9: 1SS389, Diode_SMD:D_SOD-523, symbol Device:D_Schottky_Small
- added D27: KBD_Amber, LED_SMD:LED_1206_3216Metric, symbol Mega IIe Rev3 Symbols:D_1206
- added R87, R88: 100k, Resistor_SMD:R_0603_1608Metric, symbol Device:R_Small
- added R91: 1k, Resistor_SMD:R_0805_2012Metric, symbol Mega IIe Rev3 Symbols:R_0805_1
- R26, R51: value 1K -> 4k7
- R80: value 470 -> 1k
Connections:
- net +5V_2040: now also D27.2 (A)
- net GND: now also R87.2, R88.2
- net SW0_OAPL: now also D26.1 (K), R88.1; no longer U33.6
- net SW1_CAPL: now also D9.1 (K), R87.1; no longer U31.6
- net at Q10.3 (C), R80.2: now also R91.2
- new net: D27.1 (K), R91.1
- new net: D9.2 (A), U31.6
- new net: D26.2 (A), U33.6
Other:
- moved on the sheet: C36, C41, C57, C6, J14, J21, R24, R25, U16
