File: kicad files/gd rev3b/video.kicad_sch (KiCad schematic)
At the start: 50 parts, among them J17 VGA_Micro, J18 vga_SWD, J22 L77HDE15SD1CH4F, SW6 VGA Boot Sel, SW7 VGA RESET, U19 W25Q128JVS, U22 74HCT245, U23 RP2040, U24 74LVC2G04, Y2 ECS-120-18-33-JEM-TR

Commit message: Schematic changes for #52, #50, #70, #51, #61, #69, #71
Parts:
- D11: value D_1206 -> VID_Amber
- R36: value R_0805 -> 1k
Changed lines of the file:
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@@
   (symbol (lib_id "Mega IIe Rev3 Symbols:D_1206") (at 275.59 96.52 90) (unit 1)
     (in_bom yes) (on_board yes) (dnp no) (fields_autoplaced)
-    (property "Reference" "D11" (at 278.13 95.2499 90)
+    (property "Reference" "D11" (at 278.13 95.25 90)
       (effects (font (size 1.27 1.27)) (justify right))
     )
-    (property "Value" "D_1206" (at 278.13 97.7899 90)
+    (property "Value" "VID_Amber" (at 278.13 97.79 90)
       (effects (font (size 1.27 1.27)) (justify right))
     )
@@
   (symbol (lib_id "Mega IIe Rev3 Symbols:R_0805") (at 275.59 88.9 0) (unit 1)
     (in_bom yes) (on_board yes) (dnp no) (fields_autoplaced)
-    (property "Reference" "R36" (at 278.13 87.6299 0)
-      (effects (font (size 1.27 1.27)) (justify left))
-    )
-    (property "Value" "R_0805" (at 278.13 90.1699 0)
+    (property "Reference" "R36" (at 278.13 87.63 0)
+      (effects (font (size 1.27 1.27)) (justify left))
+    )
+    (property "Value" "1k" (at 278.13 90.17 0)
       (effects (font (size 1.27 1.27)) (justify left))
     )
@@
     )
   )
-  (symbol (lib_name "+5V_2040_1") (lib_id "My Library:+5V_2040") (at 60.96 65.405 0) (unit 1)
+  (symbol (lib_id "My Library:+5V_2040") (at 60.96 65.405 0) (unit 1)
     (in_bom yes) (on_board yes) (dnp no)
     (property "Reference" "#PWR0389" (at 60.96 69.215 0)
