File: kicad files/gd rev3b/game_port.kicad_sch (KiCad schematic)
At the start: 47 parts, among them J11 Game Port, J23 Game-DB, Q4 BC817, Q5 BC817, Q6 BC817, Q7 BC817, U18 HCT251, U20 NE556, U21 NE556

Commit message: Schematic changes for #52, #50, #70, #51, #61, #69, #71
Parts:
- R58, R64, R66, R72: value 470 -> 4k7
Changed lines of the file:
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@@
       (effects (font (size 1.27 1.27)) (justify left))
     )
-    (property "Value" "470" (at 196.85 45.72 90)
+    (property "Value" "4k7" (at 196.85 45.72 90)
       (effects (font (size 1.27 1.27)) (justify left))
     )
@@
       (effects (font (size 1.27 1.27)) (justify left))
     )
-    (property "Value" "470" (at 229.87 45.72 90)
+    (property "Value" "4k7" (at 229.87 45.72 90)
       (effects (font (size 1.27 1.27)) (justify left))
     )
@@
       (effects (font (size 1.27 1.27)) (justify left))
     )
-    (property "Value" "470" (at 162.56 45.72 90)
+    (property "Value" "4k7" (at 162.56 45.72 90)
       (effects (font (size 1.27 1.27)) (justify left))
     )
@@
       (effects (font (size 1.27 1.27)) (justify left))
     )
-    (property "Value" "470" (at 262.89 46.99 90)
-      (effects (font (size 1.27 1.27)) (justify left))
-    )
+    (property "Value" "4k7" (at 262.89 46.99 90)
+      (effects (font (size 1.27 1.27)) (justify left))
+    )

Commit message: added no-load pads for SW2 and SW3 fixes #60
Parts:
- added R92, R93: 4k7, Resistor_SMD:R_0805_2012Metric, symbol Mega IIe Rev3 Symbols:R_0805_2
Connections:
- net +5V: now also R92.1, R93.1
- net SW2: now also R92.2
- net SW3: now also R93.2
Other:
- moved on the sheet: C83, R20
