File: kicad files/gd slot extender/gd slot extender.kicad_sch (KiCad schematic)
At the start: 11 parts, among them J1 Card Edge, J2 Debug Header, J3 Sockety Socket Sock

Commit message: rev1 ready for fab
Parts:
- removed D1, D2, D3, D4: D_1206, LED_SMD:LED_1206_3216Metric, symbol My Library:D_1206
- removed R1, R2, R3, R4: 4k7, Resistor_SMD:R_0805_2012Metric_Pad1.20x1.40mm_HandSolder, symbol My Library:R_0805
- added JP1: Jumper_2_Bridged, Jumper:SolderJumper-2_P1.3mm_Bridged_RoundedPad1.0x1.5mm, symbol Jumper:Jumper_2_Bridged
Connections:
- net NC: now reaches J2.19
- net NC: now also J1.19, JP1.2 (B)
- net at J3.19: now also JP1.1 (A)
- no-connect marks 3 -> 0
Other:
- moved on the sheet: J2, J3
